File: vibr.kicad_pcb (KiCad board)
At the start: 2 copper layers, 15 x 9.3 mm, 5 parts, among them J3 Conn_01x03, U3 ECH8693R-TL-W, U4 C0720B001F

Commit message: accelerometer
Other:
- board size 15 x 9.3 mm -> 15.2 x 9.3 mm
Changed lines of the file:
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@@
   (general
     (thickness 1.6)
-    (drawings 7)
+    (drawings 9)
     (tracks 45)
     (zones 0)
@@
     (solder_mask_min_width 0.25)
     (aux_axis_origin 0 0)
-    (visible_elements FFFFFF7F)
+    (visible_elements 7FFFFFFF)
     (pcbplotparams
       (layerselection 0x010fc_ffffffff)
@@
     )
   )
+  (gr_line (start 130.45 116.39) (end 130.45 117.25) (layer Edge.Cuts) (width 0.05))
+  (gr_line (start 130.440027 108.950013) (end 130.440027 107.92) (layer Edge.Cuts) (width 0.05))
+  (gr_arc (start 130.45 112.67) (end 130.45 116.39) (angle -180.1536076) (layer Edge.Cuts) (width 0.05))
   (gr_text GND (at 120.46 114.08 90) (layer F.SilkS)
     (effects (font (size 0.5 0.5) (thickness 0.125)))
@@
   )
   (gr_line (start 119 107.92) (end 118.98 117.25) (layer Edge.Cuts) (width 0.05))
-  (gr_line (start 118.98 117.25) (end 133.99 117.25) (layer Edge.Cuts) (width 0.05))
-  (gr_line (start 134 107.92) (end 133.99 117.25) (layer Edge.Cuts) (width 0.05))
-  (gr_line (start 119 107.92) (end 134 107.92) (layer Edge.Cuts) (width 0.05))
+  (gr_line (start 118.98 117.25) (end 130.45 117.25) (layer Edge.Cuts) (width 0.05))
+  (gr_line (start 119 107.92) (end 130.440027 107.92) (layer Edge.Cuts) (width 0.05))
   (via (at 123.81 110.72) (size 0.8) (drill 0.4) (layers F.Cu B.Cu) (net 1))
   (segment (start 121.750001 110.925001) (end 121.94 110.735002) (width 0.25) (layer F.Cu) (net 1))
