File: pwr.sch (KiCad schematic (older format))
At the start: 13 parts, among them J6 Conn_01x02, J7 Conn_01x05, Q2 FDC6420C, U5 SGM2036_UTDFN, U7 SGM40561

Commit message: v.01 power board PCB
Parts:
- removed D1: ZLLS410, Diodes_SMD:D_SOD-323, symbol _semi:DIODE
- removed J6: Conn_01x02, my-fp-library:Battery Pads 3x3, symbol Connector_Generic:Conn_01x02
- removed J7: Conn_01x05, Pin_Headers:Pin_Header_Straight_1x05_Pitch2.54mm, symbol Connector_Generic:Conn_01x05
- removed Q2: FDC6420C, TO_SOT_Packages_SMD:SuperSOT-6, symbol mosfet:FDC6420C
- removed U5: SGM2036_UTDFN, TO_SOT_Packages_SMD:SOT-23-5, symbol Power_Management:SGM2036_UTDFN
- removed U7: SGM40561, Housings_DFN_QFN:TDFN-2x2-8L, symbol Power_Management:SGM40561
- added C9: 10uF, Capacitors_SMD:C_0805_HandSoldering, symbol Device:C_Small
- added D1: ORANGE, LEDs:LED_0805, symbol Device:LED
- added D2: GREEN, LEDs:LED_0805, symbol Device:LED
- added J6: CONN_01X05, Pin_Headers:Pin_Header_Straight_1x05_Pitch1.27mm, symbol nrf-rescue:CONN_01X05-conn
- added P1: BATT, my-fp-library:Battery Pads 3x3, symbol nrf-rescue:CONN_01X02-conn
- added R14: 100K, Resistors_SMD:R_0805_HandSoldering, symbol Device:R
- added R15: 1K, Resistors_SMD:R_0805_HandSoldering, symbol Device:R
- added R16: 10K, Resistors_SMD:R_0805_HandSoldering, symbol Device:R
- added U5: MIC5219-3.3YM5, TO_SOT_Packages_SMD:SOT-23-5, symbol Regulator_Linear:MIC5219-3.3YM5
- added U7: MCP73871-xxI_ML, Housings_DFN_QFN:QFN-20-1EP_4x4mm_Pitch0.5mm, symbol nrf-rescue:MCP73871-xxI_ML-microchip
- C3, C7: value 1uF -> 470pF
- C6: value 0.1uF -> 470pF
- R4, R5: value 100K -> 1K; footprint Resistors_SMD:R_0805 -> Resistors_SMD:R_0805_HandSoldering
- R6: value 3M -> 270K; footprint Resistors_SMD:R_0805 -> Resistors_SMD:R_0805_HandSoldering
- R7: value 301K -> 100K; footprint Resistors_SMD:R_0805 -> Resistors_SMD:R_0805_HandSoldering
Connections:
- net labels added: PWR_SENSE, STAT, VBUS
- net labels removed: CHG, PPR, VIN
- wire segments 62 -> 80
Other:
- note added: "Charge Rate = 1000V/PROG1\n1.0K = 1000mA\n2.0K = 500mA"
- note removed: "BATT"
- note removed: "Single-cell Li-Ion battery charger"
