File: pwr.sch (KiCad schematic (older format))
At the start: 17 parts, among them J6 CONN_01X05, P1 BATT, U5 MIC5219-3.3YM5, U7 MCP73871-xxI_ML

Commit message: update for power footprint
Parts:
- J6: footprint Pin_Headers:Pin_Header_Straight_1x05_Pitch1.27mm -> Pin_Headers:Pin_Header_Straight_1x05_Pitch2.54mm
Changed lines of the file:
@@
 F 0 "J6" H 1719 2425 50  0000 C CNN
 F 1 "CONN_01X05" H 1719 2516 50  0000 C CNN
-F 2 "Pin_Headers:Pin_Header_Straight_1x05_Pitch1.27mm" H 1800 2850 50  0001 C CNN
+F 2 "Pin_Headers:Pin_Header_Straight_1x05_Pitch2.54mm" H 1800 2850 50  0001 C CNN
 F 3 "" H 1800 2850 50  0001 C CNN
 	1    1800 2850

Commit message: Initial
Parts:
- C3, C6, C7: footprint Capacitors_SMD:C_0805 -> Capacitors_SMD:C_0603_HandSoldering
- C9: footprint Capacitors_SMD:C_0805_HandSoldering -> Capacitors_SMD:C_0603_HandSoldering
- R14, R15, R16, R4, R5, R6, R7: footprint Resistors_SMD:R_0805_HandSoldering -> Resistors_SMD:R_0603_HandSoldering
Changed lines of the file:
@@
 $Descr A4 11693 8268
 encoding utf-8
-Sheet 3 5
+Sheet 2 3
 Title ""
 Date ""
@@
 F 0 "R16" V 7130 3750 50  0000 C CNN
 F 1 "10K" V 7050 3750 50  0000 C CNN
-F 2 "Resistors_SMD:R_0805_HandSoldering" V 6980 3750 50  0001 C CNN
+F 2 "Resistors_SMD:R_0603_HandSoldering" V 6980 3750 50  0001 C CNN
 F 3 "" H 7050 3750 50  0000 C CNN
 	1    7050 3750
@@
 F 0 "R6" V 4480 2650 50  0000 C CNN
 F 1 "270K" V 4400 2650 50  0000 C CNN
-F 2 "Resistors_SMD:R_0805_HandSoldering" V 4330 2650 50  0001 C CNN
+F 2 "Resistors_SMD:R_0603_HandSoldering" V 4330 2650 50  0001 C CNN
 F 3 "" H 4400 2650 50  0000 C CNN
 	1    4400 2650
@@
 F 0 "R7" V 4480 3050 50  0000 C CNN
 F 1 "100K" V 4400 3050 50  0000 C CNN
-F 2 "Resistors_SMD:R_0805_HandSoldering" V 4330 3050 50  0001 C CNN
+F 2 "Resistors_SMD:R_0603_HandSoldering" V 4330 3050 50  0001 C CNN
 F 3 "" H 4400 3050 50  0000 C CNN
 	1    4400 3050
@@
 F 0 "R5" V 4030 3050 50  0000 C CNN
 F 1 "1K" V 3950 3050 50  0000 C CNN
-F 2 "Resistors_SMD:R_0805_HandSoldering" V 3880 3050 50  0001 C CNN
+F 2 "Resistors_SMD:R_0603_HandSoldering" V 3880 3050 50  0001 C CNN
 F 3 "" H 3950 3050 50  0000 C CNN
 	1    3950 3050
@@
 F 0 "R4" V 3680 3050 50  0000 C CNN
 F 1 "1K" V 3600 3050 50  0000 C CNN
-F 2 "Resistors_SMD:R_0805_HandSoldering" V 3530 3050 50  0001 C CNN
+F 2 "Resistors_SMD:R_0603_HandSoldering" V 3530 3050 50  0001 C CNN
 F 3 "" H 3600 3050 50  0000 C CNN
 	1    3600 3050
@@
 F 0 "C9" H 7910 3470 50  0000 L CNN
 F 1 "10uF" H 7910 3320 50  0000 L CNN
-F 2 "Capacitors_SMD:C_0805_HandSoldering" H 7900 3400 50  0001 C CNN
+F 2 "Capacitors_SMD:C_0603_HandSoldering" H 7900 3400 50  0001 C CNN
 F 3 "" H 7900 3400 50  0000 C CNN
 	1    7900 3400
@@
 F 0 "R15" V 6930 3750 50  0000 C CNN
 F 1 "1K" V 6850 3750 50  0000 C CNN
-F 2 "Resistors_SMD:R_0805_HandSoldering" V 6780 3750 50  0001 C CNN
+F 2 "Resistors_SMD:R_0603_HandSoldering" V 6780 3750 50  0001 C CNN
 F 3 "" H 6850 3750 50  0000 C CNN
 	1    6850 3750
@@
 F 0 "R14" V 6730 3750 50  0000 C CNN
 F 1 "100K" V 6650 3750 50  0000 C CNN
-F 2 "Resistors_SMD:R_0805_HandSoldering" V 6580 3750 50  0001 C CNN
+F 2 "Resistors_SMD:R_0603_HandSoldering" V 6580 3750 50  0001 C CNN
 F 3 "" H 6650 3750 50  0000 C CNN
 	1    6650 3750
@@
 F 0 "C3" H 3150 6200 50  0000 L CNN
 F 1 "470pF" H 3000 6300 50  0000 L CNN
-F 2 "Capacitors_SMD:C_0805" H 3050 6200 50  0001 C CNN
+F 2 "Capacitors_SMD:C_0603_HandSoldering" H 3050 6200 50  0001 C CNN
 F 3 "" H 3050 6200 50  0000 C CNN
 	1    3050 6200
@@
 F 0 "C6" H 3500 6200 50  0000 L CNN
 F 1 "470pF" H 3350 6300 50  0000 L CNN
-F 2 "Capacitors_SMD:C_0805" H 3400 6200 50  0001 C CNN
+F 2 "Capacitors_SMD:C_0603_HandSoldering" H 3400 6200 50  0001 C CNN
 F 3 "" H 3400 6200 50  0000 C CNN
 	1    3400 6200
@@
 F 0 "C7" H 3800 6200 50  0000 L CNN
 F 1 "470pF" H 3650 6300 50  0000 L CNN
-F 2 "Capacitors_SMD:C_0805" H 3700 6200 50  0001 C CNN
+F 2 "Capacitors_SMD:C_0603_HandSoldering" H 3700 6200 50  0001 C CNN
 F 3 "" H 3700 6200 50  0000 C CNN
 	1    3700 6200
