File: 240x240_display.sch (KiCad schematic (older format))
At the start: 8 parts, among them J1 Conn_02x12_Counter_Clockwise, J5 Conn_01x09_Male, Q1 BSS138

Commit message: Power board PCB
Parts:
- removed Q1: BSS138, TO_SOT_Packages_SMD:SOT-23, symbol Transistor_FET:BSS138
- added Q1: FDC6420C, TO_SOT_Packages_SMD:SOT-666, symbol mosfet:FDC6420C
Changed lines of the file:
@@
 Wire Wire Line
 	5450 3800 5450 3650
-$Comp
-L Transistor_FET:BSS138 Q1
-U 1 1 5DA4FE84
-P 5900 4100
-F 0 "Q1" H 6106 4146 50  0000 L CNN
-F 1 "BSS138" H 6106 4055 50  0000 L CNN
-F 2 "TO_SOT_Packages_SMD:SOT-23" H 6100 4025 50  0001 L CIN
-F 3 "https://www.fairchildsemi.com/datasheets/BS/BSS138.pdf" H 5900 4100 50  0001 L CNN
-	1    5900 4100
-	1    0    0    -1
-$EndComp
 Wire Wire Line
 	5450 4100 5700 4100
@@
 Wire Wire Line
 	3700 5550 3700 5750
+$Comp
+L mosfet:FDC6420C Q1
+U 1 1 5DA8A9CF
+P 5900 4100
+F 0 "Q1" H 6091 4146 50  0000 L CNN
+F 1 "FDC6420C" H 6091 4055 50  0000 L CNN
+F 2 "TO_SOT_Packages_SMD:SOT-666" H 6100 4025 50  0001 L CNN
+F 3 "http://www.irf.com/product-info/datasheets/data/irf7309ipbf.pdf" H 5900 4100 50  0001 L CNN
+	1    5900 4100
+	1    0    0    -1
+$EndComp
 $EndSCHEMATC

Commit message: Build power board
Parts:
- Q1: footprint TO_SOT_Packages_SMD:SOT-666 -> TO_SOT_Packages_SMD:SuperSOT-6
Changed lines of the file:
@@
 F 0 "Q1" H 6091 4146 50  0000 L CNN
 F 1 "FDC6420C" H 6091 4055 50  0000 L CNN
-F 2 "TO_SOT_Packages_SMD:SOT-666" H 6100 4025 50  0001 L CNN
+F 2 "TO_SOT_Packages_SMD:SuperSOT-6" H 6100 4025 50  0001 L CNN
 F 3 "http://www.irf.com/product-info/datasheets/data/irf7309ipbf.pdf" H 5900 4100 50  0001 L CNN
 	1    5900 4100

Commit message: Circular Display
Parts:
- J1: footprint Socket_Strips:Socket_Strip_Straight_2x12_Pitch1.27mm_SMD -> SMD_Packages:DF37B-24DP-0.4V(51)
Changed lines of the file:
@@
 $Descr A4 11693 8268
 encoding utf-8
-Sheet 5 5
+Sheet 5 6
 Title ""
 Date ""
@@
 F 0 "J1" H 3700 4567 50  0000 C CNN
 F 1 "Conn_02x12_Counter_Clockwise" H 3700 4750 50  0000 C CNN
-F 2 "Socket_Strips:Socket_Strip_Straight_2x12_Pitch1.27mm_SMD" H 3650 3850 50  0001 C CNN
+F 2 "SMD_Packages:DF37B-24DP-0.4V(51)" H 3650 3850 50  0001 C CNN
 F 3 "~" H 3650 3850 50  0001 C CNN
 	1    3650 3850
