File: nrf.kicad_pcb (KiCad board)
At the start: 4 copper layers, 50 parts, among them IC1 BMA423, IC2 113990582, J2 Conn_01x05, J7 Conn_01x12, P1 BATT, Q1 SI3139K, Q2 MGSF1N02L, Q3 SI3139K, Q4 SI3139K, SW1 UP, SW2 MID, SW3 BACK, SW4 DWN, U2 C0720B001F, U3 MCP73871-xxI_ML, U4 MIC5219-3.3YM5

Commit message: Layout board
Parts:
- removed P1: BATT, my-fp-library:Battery Pads 3x3
- added C13: 4.7uF, Capacitors_SMD:C_0603_HandSoldering, F.Cu at (141.6, 95.2)
- added SW5: BACK, my-fp-library:Tact_SW_3x6x3.5, F.Cu at (124.0, 121.0)
- added TP1: TestPoint, Measurement_Points:Measurement_Point_Square-SMD-Pad_Big, F.Cu at (135.2, 92.2)
- added TP2: TestPoint, Measurement_Points:Measurement_Point_Square-SMD-Pad_Big, F.Cu at (142.2, 92.2)
- added TP3: TestPoint BATT GND, Measurement_Points:Measurement_Point_Square-SMD-Pad_Big, F.Cu at (119.2, 78.6)
- added TP4: TestPoint BATT GND, Measurement_Points:Measurement_Point_Square-SMD-Pad_Big, F.Cu at (123.7, 78.6)
- added U1: GD25Q16, SMD_Packages:USON8-4x3, F.Cu at (129.4, 102.3)
- added X1: 32.768, Crystals:Crystal_SMD_EuroQuartz_EQ161-2pin_3.2x1.5mm_HandSoldering, F.Cu at (142.6, 115.2)
- C1, C10: value 22pF -> 9pF
- J7: moved to B.Cu
- SW3: value BACK -> DOWN
- SW4: value DWN -> RESET; footprint my-fp-library:Tact_SW_3x6x3.5 -> Buttons_Switches_SMD:SW_SPST_B3U-1000P
- moved R13 64.4 mm to (140.2, 119.4), turned to 90 degrees
- moved R2 63.4 mm to (130.7, 126.4)
- moved R10 59.8 mm to (141.4, 119.4), turned to 90 degrees
- moved Q4 59.2 mm to (130.9, 118.7)
- moved Q3 59.2 mm to (130.8, 122.0), turned to 270 degrees
- moved D2 59.0 mm to (131.4, 92.8)
- moved Q1 56.2 mm to (127.5, 118.7), turned to 180 degrees
- moved J7 54.7 mm to (139.5, 123.0)
- moved R4 53.0 mm to (129.3, 96.0)
- moved Q2 52.4 mm to (143.1, 128.4)
- moved D1 51.6 mm to (129.3, 94.4)
- moved R16 48.6 mm to (133.8, 95.0), turned to 180 degrees
- moved U4 47.5 mm to (146.4, 95.5)
- moved C3 46.7 mm to (141.6, 99.2)
- moved U3 46.4 mm to (138.4, 97.2), turned to 270 degrees
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Connections:
- net Net-(C3-Pad1) renamed /BATT
- IC1 pad 5: (no net) -> /INT1
- IC1 pad 6: (no net) -> /INT2
- IC2 pad 25: (no net) -> /BTN_4
- IC2 pad 41: (no net) -> /QSPI_DATA0
- IC2 pad 42: (no net) -> /QSPI_SCK
- IC2 pad 43: (no net) -> /QSPI_DATA3
- IC2 pad 44: (no net) -> /QSPI_CS
- IC2 pad 45: (no net) -> /QSPI_DATA2
- IC2 pad 48: (no net) -> /INT1
- IC2 pad 49: (no net) -> /INT2
Routing:
- net /QSPI_DATA2: track 0.00 -> 10.5 mm, vias 0 -> 2
- net /QSPI_DATA3: track 0.00 -> 5.11 mm
- net /QSPI_CS: track 0.00 -> 4.74 mm
- net /QSPI_SCK: track 0.00 -> 4.17 mm
- net /BATT: track 0.00 -> 2.81 mm
- net /VOUT: track 0.00 -> 2.36 mm
- net /QSPI_DATA0: track 0.00 -> 1.93 mm

Commit message: Layout board
Parts:
- removed D2: GREEN, LEDs:LED_0805
- removed R5: 1K, Resistors_SMD:R_0603_HandSoldering
- TP3: moved to B.Cu
- moved J2 37.8 mm to (127.7, 98.6), turned to 315 degrees
- moved TP4 32.1 mm to (151.0, 95.5)
- moved TP3 23.8 mm to (138.7, 92.2)
- moved R18 20.5 mm to (136.4, 126.3), turned to 270 degrees
- moved R19 18.7 mm to (138.4, 126.3), turned to 270 degrees
- moved R1 16.9 mm to (146.0, 113.8)
- moved Q2 12.9 mm to (147.0, 116.1)
- moved R17 12.3 mm to (144.7, 116.4), turned to 90 degrees
- moved R3 11.4 mm to (131.7, 122.6)
- moved R13 10.4 mm to (130.3, 122.6)
- moved R8 10.4 mm to (137.2, 116.6)
- moved R2 10.2 mm to (133.4, 116.6)
- moved R10 8.90 mm to (133.1, 122.6)
- moved C2 7.77 mm to (125.9, 117.8), turned to 270 degrees
- moved C11 7.73 mm to (127.1, 117.7), turned to 270 degrees
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Connections:
- IC2 pad 12: (no net) -> /LIGHT3
- IC2 pad 14: (no net) -> /LIGHT1
- IC2 pad 16: /LIGHT1 -> (no net)
- IC2 pad 19: /LIGHT2 -> (no net)
- IC2 pad 20: (no net) -> /BTN_3
- IC2 pad 22: /BTN_1 -> /BTN_2
- IC2 pad 23: /BTN_2 -> (no net)
- IC2 pad 24: /BTN_3 -> /BTN_1
- IC2 pad 4: (no net) -> /LIGHT2
- IC2 pad 46: (no net) -> /QSPI_DATA1
- IC2 pad 56: /PWR_SENSE -> (no net)
- IC2 pad 57: /PWR_STAT -> (no net)
- IC2 pad 8: /LIGHT3 -> (no net)
- R4 pad 2: /PWR_SENSE -> Net-(R4-Pad2)
- U1 pad 2: (no net) -> /QSPI_DATA1
- U3 pad 7: /PWR_STAT -> (no net)
- U3 pad 8: /PWR_SENSE -> Net-(R4-Pad2)
Routing:
- net +3.3: track 0.00 -> 23.3 mm
- net /XL1: track 0.00 -> 9.26 mm
- net /VOUT: track 2.36 -> 11.1 mm
- net +5: track 0.00 -> 8.31 mm
- net /XL2: track 0.00 -> 8.28 mm
- net /SWDIO: track 0.00 -> 6.33 mm
- net /SWDCLK: track 0.00 -> 5.55 mm
- net /QSPI_DATA1: track 0.00 -> 4.30 mm
- net Net-(Q3-Pad3): track 0.00 -> 4.02 mm
- net Net-(R15-Pad1): track 0.00 -> 3.79 mm
- net Net-(D4-Pad2): track 0.00 -> 3.62 mm
- net Net-(Q2-Pad1): track 0.00 -> 3.39 mm
- net /LEDK: track 0.00 -> 2.90 mm
- net (GND): track 0.00 -> 2.85 mm
- net Net-(Q1-Pad3): track 0.00 -> 2.78 mm
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- added copper zone on B.Cu, net (GND)
Other:
- board outline added: 42 x 42 mm

Commit message: Layout board
Parts:
- removed D1: ORANGE, LEDs:LED_0805
- added TP5: TestPoint, Measurement_Points:Measurement_Point_Square-SMD-Pad_Small, F.Cu at (127.9, 95.8)
- R4: value 1K -> 10K
- moved TP2 2.20 mm to (140.0, 92.2)
- moved TP3 1.30 mm to (140.0, 92.2)
- moved R16 1.10 mm to (134.9, 95.1)
- moved C5 1.10 mm to (151.6, 104.5)
- moved R4 0.70 mm to (133.8, 96.5)
Connections:
- IC2 pad 56: (no net) -> /PWR_CHRGING
- R4 pad 1: Net-(D1-Pad1) -> +5
- R4 pad 2: Net-(R4-Pad2) -> /PWR_CHRGING
- U3 pad 8: Net-(R4-Pad2) -> /PWR_CHRGING
Routing:
- net (GND): track 2.85 -> 29.0 mm, vias 0 -> 18
- net /PWR_CHRGING: track 0.00 -> 7.27 mm, vias 0 -> 2
- net /VOUT: track 11.1 -> 14.4 mm, vias 0 -> 2
- net Net-(R4-Pad2): track 2.49 -> 0.00 mm
- net +5: track 8.31 -> 6.06 mm
- net Net-(D1-Pad1): track 1.50 -> 0.00 mm
- net Net-(R16-Pad1): track 2.46 -> 1.34 mm
- added copper zone on F.Cu, net +3.3
- added copper zone on F.Cu, net +5

Commit message: Layout board
Parts:
- moved R6 7.87 mm to (139.2, 95.0)
- moved R12 7.78 mm to (148.7, 107.3), turned to 90 degrees
- moved IC1 7.07 mm to (145.8, 106.2)
- moved C5 7.07 mm to (145.3, 107.8)
- moved C7 6.96 mm to (146.9, 99.2)
- moved R11 5.98 mm to (146.8, 102.8), turned to 0 degrees
- moved R7 5.46 mm to (142.9, 95.0), turned to 0 degrees
- moved C4 5.28 mm to (146.6, 104.0), turned to 0 degrees
- moved C9 4.57 mm to (146.9, 98.0)
- moved R15 4.02 mm to (140.8, 102.0), turned to 0 degrees
- moved C13 1.00 mm to (141.7, 96.2)
- moved U3 1.00 mm to (138.4, 98.2)
- moved C3 1.00 mm to (141.6, 100.2)
- moved R14 1.00 mm to (136.8, 102.0)
- moved R16 1.00 mm to (134.9, 96.1)
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Routing:
- net +5: track 6.06 -> 30.2 mm, vias 0 -> 2
- net (GND): track 29.0 -> 47.5 mm, vias 18 -> 35
- net /LIGHT1: track 2.68 -> 9.59 mm
- net /LIGHT3: track 1.42 -> 6.66 mm
- net /LIGHT2: track 1.44 -> 5.75 mm
- net /VOUT: track 14.4 -> 11.6 mm, vias 2 -> 0
- net /PWR_CHRGING: track 7.27 -> 9.88 mm
- net Net-(R6-Pad2): track 1.35 -> 3.74 mm
- net /SCL: track 0.00 -> 2.03 mm
- net Net-(R15-Pad1): track 3.79 -> 2.32 mm
- net +3.3: track 23.8 -> 24.6 mm
- removed copper zone on F.Cu, net +5

Commit message: Layout board
Parts:
- moved SW4 21.1 mm to (125.5, 97.5), turned to 55 degrees
- moved C5 6.13 mm to (148.6, 102.6), turned to 180 degrees
- moved R12 5.44 mm to (145.2, 103.1), turned to 270 degrees
- moved R11 5.34 mm to (148.5, 107.8), turned to 180 degrees
- moved IC1 2.94 mm to (148.1, 104.2), turned to 0 degrees
- moved TP5 2.82 mm to (130.2, 94.1)
- moved C4 2.51 mm to (147.3, 106.4), turned to 180 degrees
Routing:
- net /BTN_1: track 0.00 -> 31.2 mm, vias 0 -> 2
- net /BTN_3: track 0.00 -> 28.1 mm, vias 0 -> 2
- net /BTN_2: track 0.00 -> 24.9 mm, vias 0 -> 2
- net (GND): track 47.5 -> 59.3 mm
- net +3.3: track 24.6 -> 29.6 mm, vias 0 -> 1
- net /SDA: track 0.00 -> 4.09 mm, vias 0 -> 1
- net /SPI_RESET: track 0.00 -> 2.25 mm, vias 0 -> 1
- net /SPI_CS: track 0.00 -> 2.05 mm, vias 0 -> 1
- net /SCL: track 2.03 -> 3.11 mm, vias 0 -> 1
Other:
- copper layers 4 -> 2

Commit message: Layout board
Parts:
- moved D4 3.09 mm to (151.0, 116.2), turned to 90 degrees
- moved R11 2.93 mm to (150.9, 106.2), turned to 90 degrees
- moved C8 2.06 mm to (143.8, 126.3)
- moved J7 2.06 mm to (141.1, 124.3)
- moved R19 1.66 mm to (139.0, 127.8)
- moved R18 1.55 mm to (136.8, 127.8)
- moved R1 1.39 mm to (146.8, 112.7)
- moved C3 1.30 mm to (142.9, 100.2)
- moved C13 1.30 mm to (142.9, 96.2)
- moved Q2 1.24 mm to (147.9, 115.2)
- moved C4 1.19 mm to (147.8, 107.5)
- moved R17 1.18 mm to (145.4, 115.5)
- moved C5 1.15 mm to (148.2, 101.5)
- moved R16 1.10 mm to (133.8, 96.0)
- moved U2 0.75 mm to (148.8, 125.0)
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Routing:
- net /SDA: track 4.09 -> 25.2 mm, vias 1 -> 4
- net /SCL: track 3.11 -> 18.4 mm, vias 1 -> 4
- net /BATT: track 2.81 -> 4.23 mm
- net /SPI_CS: track 2.05 -> 3.23 mm
- net Net-(R16-Pad1): track 1.34 -> 2.48 mm
- net /SPI_RESET: track 2.25 -> 3.39 mm
- net Net-(D4-Pad2): track 3.62 -> 4.76 mm
- net +5: track 30.2 -> 31.2 mm
- net /QSPI_DATA2: track 10.5 -> 11.4 mm
- net /VOUT: track 11.6 -> 12.6 mm
- net +3.3: track 29.6 -> 30.4 mm
- net (GND): track 59.3 -> 59.0 mm, vias 35 -> 33
Other:
- rule solder_mask_min_width: 0.25 -> 0.101

Commit message: Layout board
Parts:
- Q1, Q3, Q4: footprint TO_SOT_Packages_SMD:SOT-23 -> TO_SOT_Packages_SMD:SOT-723_Handsoldering
- moved R2 21.3 mm to (113.6, 124.5)
- moved C2 21.3 mm to (106.1, 125.6)
- moved Q4 21.3 mm to (110.1, 126.8)
- moved R13 21.3 mm to (110.5, 130.4)
- moved R9 21.3 mm to (109.8, 124.5)
- moved C11 21.3 mm to (107.3, 125.5)
- moved Q3 21.3 mm to (116.7, 126.8)
- moved R10 21.3 mm to (113.3, 130.4)
- moved Q1 21.3 mm to (113.4, 126.8)
- moved R3 21.3 mm to (111.9, 130.4)
- moved R8 21.3 mm to (117.4, 124.5)
- moved C5 6.54 mm to (153.3, 105.6), turned to 90 degrees
- moved R12 6.52 mm to (151.8, 102.6), turned to 180 degrees
- moved R11 5.14 mm to (146.1, 107.8), turned to 0 degrees
- moved IC1 2.77 mm to (150.6, 105.5), turned to 270 degrees
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Connections:
- IC2 pad 10: (no net) -> /SPI_DC
- IC2 pad 13: (no net) -> /LIGHT2
- IC2 pad 25: /BTN_4 -> (no net)
- IC2 pad 26: /MOTOR_PWM -> /INT2
- IC2 pad 27: /SCL -> (no net)
- IC2 pad 29: /SDA -> (no net)
- IC2 pad 3: (no net) -> /SPI_RESET
- IC2 pad 31: (no net) -> /INT1
- IC2 pad 34: (no net) -> /SDA
- IC2 pad 35: (no net) -> /SCL
- IC2 pad 36: /SPI_SCK -> (no net)
- IC2 pad 37: /SPI_MOSI -> (no net)
- IC2 pad 38: /SPI_CS -> (no net)
- IC2 pad 39: /SPI_DC -> (no net)
- IC2 pad 4: /LIGHT2 -> /SPI_MOSI
- IC2 pad 45: /QSPI_DATA2 -> (no net)
- IC2 pad 47: /SPI_RESET -> (no net)
- IC2 pad 48: /INT1 -> /QSPI_DATA2
- IC2 pad 49: /INT2 -> /MOTOR_PWM
- IC2 pad 5: (no net) -> /BTN_4
- IC2 pad 6: (no net) -> /SPI_SCK
- IC2 pad 8: (no net) -> /SPI_CS
Routing:
- net /INT1: track 0.00 -> 20.1 mm, vias 0 -> 2
- net /INT2: track 0.00 -> 19.5 mm, vias 0 -> 2
- net +3.3: track 30.4 -> 12.2 mm, vias 1 -> 2
- net /SPI_DC: track 0.00 -> 18.1 mm, vias 0 -> 1
- net /SPI_CS: track 3.23 -> 21.3 mm, vias 1 -> 2
- net /SPI_MOSI: track 0.00 -> 18.1 mm, vias 0 -> 1
- net /SPI_RESET: track 3.39 -> 21.4 mm, vias 1 -> 2
- net /SPI_SCK: track 0.00 -> 17.9 mm, vias 0 -> 1
- net /LIGHT1: track 9.59 -> 0.00 mm
- net /BTN_4: track 0.00 -> 7.84 mm
- net /QSPI_DATA2: track 11.4 -> 3.87 mm, vias 2 -> 0
- net /LIGHT3: track 6.66 -> 0.00 mm
- net /LIGHT2: track 5.75 -> 0.00 mm
- net /SDA: track 25.2 -> 20.2 mm, vias 4 -> 2
- net (GND): track 59.0 -> 54.9 mm, vias 33 -> 31
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
Commit message: More layout changes
Parts:
- removed TP5: TestPoint, Measurement_Points:Measurement_Point_Square-SMD-Pad_Small
- added C14: ??pF, Capacitors_SMD:C_0603_HandSoldering, F.Cu at (141.0, 94.5)
- added R5: 1, Resistors_SMD:R_0603_HandSoldering, F.Cu at (136.2, 94.2)
- U2: moved to B.Cu
- moved C8 51.2 mm to (174.3, 85.2)
- moved C2 49.5 mm to (146.2, 96.5), turned to 180 degrees
- moved R3 48.9 mm to (149.6, 99.2), turned to 270 degrees
- moved C11 45.9 mm to (145.1, 99.4), turned to 90 degrees
- moved R19 45.6 mm to (153.6, 84.6), turned to 0 degrees
- moved R2 45.6 mm to (151.6, 99.3), turned to 270 degrees
- moved R10 45.6 mm to (146.5, 99.2), turned to 270 degrees
- moved R13 45.3 mm to (143.6, 99.5), turned to 270 degrees
- moved R18 44.6 mm to (153.3, 86.3), turned to 0 degrees
- moved Q1 44.0 mm to (150.0, 102.5), turned to 90 degrees
- moved Q4 42.0 mm to (144.2, 102.5), turned to 90 degrees
- moved R9 40.8 mm to (142.1, 99.5), turned to 270 degrees
- moved R8 39.7 mm to (148.0, 99.2), turned to 270 degrees
- moved Q3 39.0 mm to (147.1, 102.5), turned to 90 degrees
- moved SW2 35.5 mm to (124.0, 110.0), turned to 90 degrees
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Connections:
- IC1 pad 10: (no net) -> Net-(IC1-Pad10)
- IC1 pad 11: (no net) -> Net-(IC1-Pad11)
- IC1 pad 4: (no net) -> Net-(IC1-Pad4)
- IC2 pad 11: (no net) -> Net-(IC2-Pad11)
- IC2 pad 16: (no net) -> Net-(IC2-Pad16)
- IC2 pad 19: (no net) -> /SDA
- IC2 pad 20: /BTN_3 -> /BTN_1
- IC2 pad 21: (no net) -> /SCL
- IC2 pad 23: (no net) -> Net-(IC2-Pad23)
- IC2 pad 24: /BTN_1 -> /BTN_3
- IC2 pad 25: (no net) -> Net-(IC2-Pad25)
- IC2 pad 27: (no net) -> Net-(IC2-Pad27)
- IC2 pad 29: (no net) -> /MOTOR_PWM
- IC2 pad 34: /SDA -> Net-(IC2-Pad34)
- IC2 pad 35: /SCL -> Net-(IC2-Pad35)
- IC2 pad 36: (no net) -> Net-(IC2-Pad36)
- IC2 pad 37: (no net) -> Net-(IC2-Pad37)
- IC2 pad 38: (no net) -> Net-(IC2-Pad38)
- IC2 pad 39: (no net) -> /PWR_CHRGING
- IC2 pad 45: (no net) -> Net-(IC2-Pad45)
- IC2 pad 47: (no net) -> Net-(IC2-Pad47)
- IC2 pad 49: /MOTOR_PWM -> /BTN_4
- IC2 pad 5: /BTN_4 -> Net-(IC2-Pad5)
- IC2 pad 50: (no net) -> Net-(IC2-Pad50)
- IC2 pad 52: (no net) -> Net-(IC2-Pad52)
- IC2 pad 54: (no net) -> Net-(IC2-Pad54)
- IC2 pad 56: /PWR_CHRGING -> Net-(IC2-Pad56)
- IC2 pad 57: (no net) -> Net-(IC2-Pad57)
- IC2 pad 58: (no net) -> Net-(IC2-Pad58)
- IC2 pad 59: (no net) -> Net-(IC2-Pad59)
- IC2 pad 60: (no net) -> Net-(IC2-Pad60)
- IC2 pad 61: (no net) -> Net-(IC2-Pad61)
- IC2 pad 7: (no net) -> Net-(IC2-Pad7)
- IC2 pad 9: (no net) -> Net-(IC2-Pad9)
- J2 pad 1: +3.3 -> (GND)
- J2 pad 2: /SWDIO -> /RESET
- J2 pad 4: /RESET -> /SWDIO
- J2 pad 5: (GND) -> +3.3
- J7 pad 2: /LEDK -> Net-(J7-Pad2)
- J7 pad 3: +3.3 -> /LEDA
- R10 pad 1: /LEDK -> /LEDA
- R13 pad 1: /LEDK -> /LEDA
- R3 pad 1: /LEDK -> /LEDA
- U3 pad 6: (no net) -> Net-(U3-Pad6)
- U3 pad 7: (no net) -> Net-(U3-Pad7)
Routing:
- net /BTN_1: track 31.0 -> 0.00 mm, vias 2 -> 0
- net /BTN_3: track 28.1 -> 0.00 mm, vias 2 -> 0
- net +5: track 32.1 -> 6.47 mm, vias 2 -> 0
- net /BTN_2: track 25.0 -> 0.00 mm, vias 2 -> 0
- net /SPI_RESET: track 21.4 -> 0.00 mm, vias 2 -> 0
- net (GND): track 54.9 -> 42.0 mm, vias 31 -> 30
- net /LIGHT3: track 0.00 -> 9.47 mm
- net /MOTOR_PWM: track 0.00 -> 8.73 mm, vias 0 -> 2
- net /LIGHT2: track 0.00 -> 8.67 mm
- net /SPI_CS: track 21.3 -> 12.7 mm, vias 2 -> 1
- net /LIGHT1: track 0.00 -> 7.53 mm
- net /LEDA: track 0.00 -> 7.51 mm
- net /PWR_CHRGING: track 9.54 -> 2.51 mm, vias 2 -> 0
- net /SWDIO: track 6.33 -> 0.00 mm
- net /INT2: track 19.5 -> 13.6 mm
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Other:
- board size 42 x 42 mm -> 35.6 x 35.6 mm
