File: nrf.sch (KiCad schematic (older format))
At the start: 31 parts, among them IC2 113990582, J2 Conn_01x05, J7 Conn_01x12, Q1 SI3139K, Q2 MGSF1N02L, Q3 SI3139K, Q4 SI3139K, SW1 UP, SW2 MID, SW3 BACK, SW4 DWN, U1 GD25Q16, U2 C0720B001F, X1 32.768

Commit message: Update for accel
Parts:
- added C4, C5: 0.1uF, Capacitors_SMD:C_0603_HandSoldering, symbol Device:C_Small
- added IC1: BMA423, SamacSys_Parts:BMA423, symbol SamacSys_Parts:BMA423
- added R11, R12: 10K, Resistors_SMD:R_0603_HandSoldering, symbol Device:R_Small
- J7: footprint (none) -> my-fp-library:FPC_12x0.7mm
Connections:
- net labels added: INT1, INT2, SPI_MOSI, SPI_SCK
- net labels removed: SPI_SCL, SPI_SDA
- wire segments 152 -> 184

Commit message: Move power from sub sheet
Parts:
- added C3: 10uF, Capacitors_SMD:C_0603_HandSoldering, symbol Device:C_Small
- added C6, C7, C9: 470pF, Capacitors_SMD:C_0603_HandSoldering, symbol Device:C_Small
- added D1: ORANGE, LEDs:LED_0805, symbol Device:LED
- added D2: GREEN, LEDs:LED_0805, symbol Device:LED
- added P1: BATT, my-fp-library:Battery Pads 3x3, symbol nrf-rescue:CONN_01X02-conn
- added R14, R7: 100K, Resistors_SMD:R_0603_HandSoldering, symbol Device:R
- added R15, R4, R5: 1K, Resistors_SMD:R_0603_HandSoldering, symbol Device:R
- added R16: 10K, Resistors_SMD:R_0603_HandSoldering, symbol Device:R
- added R6: 270K, Resistors_SMD:R_0603_HandSoldering, symbol Device:R
- added U3: MCP73871-xxI_ML, Housings_DFN_QFN:QFN-20-1EP_4x4mm_Pitch0.5mm, symbol nrf-rescue:MCP73871-xxI_ML-microchip
- added U4: MIC5219-3.3YM5, TO_SOT_Packages_SMD:SOT-23-5, symbol Regulator_Linear:MIC5219-3.3YM5
Connections:
- net labels added: +5, PWR_SENSE, PWR_STAT, VOUT
- wire segments 184 -> 264
Other:
- note added: "3.3V Regulator"
- note added: "Charge Rate = 1000V/PROG1\n1.0K = 1000mA\n2.0K = 500mA"
- moved on the sheet: C1, C10, C11, C2, C4, C5, C8, D4, IC1, J7, Q1, Q2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

Commit message: Layout board
Parts:
- removed P1: BATT, my-fp-library:Battery Pads 3x3, symbol nrf-rescue:CONN_01X02-conn
- removed unit 2 of SW3
- added C13: 4.7uF, Capacitors_SMD:C_0603_HandSoldering, symbol Device:C_Small
- added SW5: BACK, my-fp-library:Tact_SW_3x6x3.5, symbol Switch:SW_DPST_x2
- added TP1, TP2: TestPoint, Measurement_Points:Measurement_Point_Square-SMD-Pad_Big, symbol Connector:TestPoint
- added TP3, TP4: TestPoint BATT GND, Measurement_Points:Measurement_Point_Square-SMD-Pad_Big, symbol Connector:TestPoint
- C1, C10: value 22pF -> 9pF
- SW3: value BACK -> DOWN
- SW4: value DWN -> RESET; footprint my-fp-library:Tact_SW_3x6x3.5 -> Buttons_Switches_SMD:SW_SPST_B3U-1000P
- U1: footprint Package_SO:SOIC-8_3.9x4.9mm_P1.27mm -> SMD_Packages:USON8-4x3; dims (none) -> 8-USON (4x3)
- X1: footprint (none) -> Crystals:Crystal_SMD_EuroQuartz_EQ161-2pin_3.2x1.5mm_HandSoldering; Digikey (none) -> https://www.digikey.com/products/en/crystals-oscillators-re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
Connections:
- net labels added: BATT
- wire segments 264 -> 271
- no-connect marks 0 -> 27
Changed lines of the file:
@@
 P 5150 1950
 F 0 "SW3" H 5150 2185 50  0000 C CNN
-F 1 "BACK" H 5150 2094 50  0000 C CNN
+F 1 "DOWN" H 5150 2094 50  0000 C CNN
 F 2 "my-fp-library:Tact_SW_3x6x3.5" H 5150 1950 50  0001 C CNN
 F 3 "" H 5150 1950 50  0001 C CNN
@@
 Wire Wire Line
 	4550 1950 4550 2300
-$Comp
-L Switch:SW_DPST_x2 SW3
-U 2 1 5EAE6769
-P 5150 2300
-F 0 "SW3" H 5150 2535 50  0000 C CNN
-F 1 "BACK" H 5150 2444 50  0000 C CNN
-F 2 "my-fp-library:Tact_SW_3x6x3.5" H 5150 2300 50  0001 C CNN
-F 3 "" H 5150 2300 50  0001 C CNN
-	2    5150 2300
-	1    0    0    -1
-$EndComp
 Wire Wire Line
 	4950 2300 4550 2300
@@
 F 0 "X1" V 1685 7100 50  0000 C CNN
 F 1 "32.768" V 1776 7100 50  0000 C CNN
-F 2 "" H 1900 7100 60  0001 C CNN
-F 3 "" H 1900 7100 60  0000 C CNN
+F 2 "Crystals:Crystal_SMD_EuroQuartz_EQ161-2pin_3.2x1.5mm_HandSoldering" H 1900 7100 60  0001 C CNN
+F 3 "https://abracon.com/Resonators/ABS07.pdf" H 1900 7100 60  0001 C CNN
+F 4 "https://www.digikey.com/products/en/crystals-oscillators-resonators/crystals/171?k=&pkeyword=&sv=0&pv537=1398&pv2082=u70+kOhms&sf=1&FV=-1%7C535%2C35%7C305379%2C-8%7C171%2C16%7C168669&quantity=&ColumnSort=0&page=1&pageSize=25" V 1900 7100 50  0001 C CNN "Digikey"
 	1    1900 7100
 	0    1    1    0
@@
 P 1650 7400
 F 0 "C1" H 1742 7446 50  0000 L CNN
-F 1 "22pF" H 1742 7355 50  0000 L CNN
+F 1 "9pF" H 1742 7355 50  0000 L CNN
 F 2 "Capacitors_SMD:C_0603_HandSoldering" H 1650 7400 50  0001 C CNN
 F 3 "~" H 1650 7400 50  0001 C CNN
@@
 P 2150 7400
 F 0 "C10" H 2242 7446 50  0000 L CNN
-F 1 "22pF" H 2242 7355 50  0000 L CNN
+F 1 "9pF" H 2242 7355 50  0000 L CNN
 F 2 "Capacitors_SMD:C_0603_HandSoldering" H 2150 7400 50  0001 C CNN
 F 3 "~" H 2150 7400 50  0001 C CNN
@@
 P 3000 7400
 F 0 "SW4" H 3000 7635 50  0000 C CNN
-F 1 "DWN" H 3000 7544 50  0000 C CNN
-F 2 "my-fp-library:Tact_SW_3x6x3.5" H 3000 7400 50  0001 C CNN
+F 1 "RESET" H 3000 7544 50  0000 C CNN
+F 2 "Buttons_Switches_SMD:SW_SPST_B3U-1000P" H 3000 7400 50  0001 C CNN
 F 3 "" H 3000 7400 50  0001 C CNN
 	1    3000 7400
@@
 F 0 "U1" H 12300 5900 50  0000 L CNN
 F 1 "GD25Q16" H 11500 5850 50  0000 L CNN
-F 2 "Package_SO:SOIC-8_3.9x4.9mm_P1.27mm" H 11950 4850 50  0001 C CNN
-F 3 "https://www.adestotech.com/wp-content/uploads/DS-AT25SF081_045.pdf" H 11950 5450 50  0001 C CNN
+F 2 "SMD_Packages:USON8-4x3" H 11950 4850 50  0001 C CNN
+F 3 "http://www.gigadevice.com/datasheet/gd25q16c/" H 11950 5450 50  0001 C CNN
+F 4 "8-USON (4x3)" H 11950 5450 50  0001 C CNN "dims"
 	1    11950 5450
 	1    0    0    -1
@@
 	5050 3300 5300 3300
 $Comp
-L nrf-rescue:CONN_01X02-conn P1
-U 1 1 5EC59A90
-P 5250 5550
-AR Path="/5EC59A90" Ref="P1"  Part="1"
-AR Path="/5C2799D2/5EC59A90" Ref="P?"  Part="1"
-AR Path="/5D08BD3C/5EC59A90" Ref="P?"  Part="1"
-F 0 "P1" H 5250 5700 50  0000 C CNN
-F 1 "BATT" V 5350 5550 50  0000 C CNN
-F 2 "my-fp-library:Battery Pads 3x3" H 5250 5550 50  0001 C CNN
-F 3 "" H 5250 5550 50  0000 C CNN
-	1    5250 5550
-	1    0    0    -1
-$EndComp
-$Comp
 L nrf-rescue:(GND)-power1 #PWR041
 U 1 1 5EC59A96
-P 5050 5750
+P 5800 7600
 AR Path="/5EC59A96" Ref="#PWR041"  Part="1"
 AR Path="/5C2799D2/5EC59A96" Ref="#PWR?"  Part="1"
 AR Path="/5D08BD3C/5EC59A96" Ref="#PWR?"  Part="1"
-F 0 "#PWR041" H 5050 5750 30  0001 C CNN
-F 1 "(GND)" H 5050 5750 30  0001 C CNN
-F 2 "" H 5050 5750 60  0000 C CNN
-F 3 "" H 5050 5750 60  0000 C CNN
-	1    5050 5750
-	1    0    0    -1
-$EndComp
-Wire Wire Line
-	5050 5600 5050 5750
+F 0 "#PWR041" H 5800 7600 30  0001 C CNN
+F 1 "(GND)" H 5800 7600 30  0001 C CNN
+F 2 "" H 5800 7600 60  0000 C CNN
+F 3 "" H 5800 7600 60  0000 C CNN
+	1    5800 7600
+	1    0    0    -1
+$EndComp
 $Comp
 L Device:R R16
@@
 	4050 4700 4350 4700
 Wire Wire Line
-	4350 4700 4550 4700
+	4350 4700 4450 4700
 Wire Wire Line
 	4050 4800 4350 4800
@@
 Text Label 3150 3550 0    50   ~ 0
 PWR_STAT
+$Comp
+L Switch:SW_DPST_x2 SW5
+U 1 1 5EC305B1
+P 5150 2300
+F 0 "SW5" H 5150 2535 50  0000 C CNN
+F 1 "BACK" H 5150 2444 50  0000 C CNN
+F 2 "my-fp-library:Tact_SW_3x6x3.5" H 5150 2300 50  0001 C CNN
+F 3 "" H 5150 2300 50  0001 C CNN
+	1    5150 2300
+	1    0    0    -1
+$EndComp
+$Comp
+L Connector:TestPoint TP1
+U 1 1 5EC905BD
+P 4500 7550
+F 0 "TP1" H 4442 7576 50  0000 R CNN
+F 1 "TestPoint" H 4442 7667 50  0000 R CNN
+F 2 "Measurement_Points:Measurement_Point_Square-SMD-Pad_Big" H 4700 7550 50  0001 C CNN
+F 3 "~" H 4700 7550 50  0001 C CNN
+	1    4500 7550
+	-1   0    0    1
+$EndComp
+$Comp
+L power:+5 #PWR048
+U 1 1 5EC91C14
+P 4500 7350
+F 0 "#PWR048" H 4500 7400 30  0001 C CNN
+F 1 "+5" H 4500 7483 50  0000 C CNN
+F 2 "" H 4500 7350 60  0000 C CNN
+F 3 "" H 4500 7350 60  0000 C CNN
+	1    4500 7350
+	1    0    0    -1
+$EndComp
+Wire Wire Line
+	4500 7350 4500 7550
+$Comp
+L Connector:TestPoint TP2
+U 1 1 5ECC59D8
+P 5250 7400
+F 0 "TP2" H 5192 7426 50  0000 R CNN
+F 1 "TestPoint" H 5192 7517 50  0000 R CNN
+F 2 "Measurement_Points:Measurement_Point_Square-SMD-Pad_Big" H 5450 7400 50  0001 C CNN
+F 3 "~" H 5450 7400 50  0001 C CNN
+	1    5250 7400
+	1    0    0    -1
+$EndComp
+Wire Wire Line
+	5250 7600 5250 7400
+$Comp
+L power:(GND) #PWR?
+U 1 1 5ECDB2CB
+P 5250 7600
+AR Path="/5DA394ED/5ECDB2CB" Ref="#PWR?"  Part="1"
+AR Path="/5ECDB2CB" Ref="#PWR049"  Part="1"
+F 0 "#PWR049" H 5250 7600 30  0001 C CNN
+F 1 "(GND)" H 5250 7600 30  0001 C CNN
+F 2 "" H 5250 7600 60  0000 C CNN
+F 3 "" H 5250 7600 60  0000 C CNN
+	1    5250 7600
+	1    0    0    -1
+$EndComp
+Wire Wire Line
+	5050 5500 5350 5500
+Text Label 5150 5500 0    50   ~ 0
+BATT
+$Comp
+L Connector:TestPoint TP3
+U 1 1 5ED057C8
+P 5800 7400
+F 0 "TP3" H 5858 7518 50  0000 L CNN
+F 1 "TestPoint BATT GND" H 5858 7427 50  0000 L CNN
+F 2 "Measurement_Points:Measurement_Point_Square-SMD-Pad_Big" H 6000 7400 50  0001 C CNN
+F 3 "~" H 6000 7400 50  0001 C CNN
+	1    5800 7400
+	1    0    0    -1
+$EndComp
+Wire Wire Line
+	5800 7400 5800 7600
+$Comp
+L Connector:TestPoint TP4
+U 1 1 5ED3082D
+P 6700 7500
+F 0 "TP4" H 6642 7526 50  0000 R CNN
+F 1 "TestPoint BATT GND" H 6642 7617 50  0000 R CNN
+F 2 "Measurement_Points:Measurement_Point_Square-SMD-Pad_Big" H 6900 7500 50  0001 C CNN
+F 3 "~" H 6900 7500 50  0001 C CNN
+	1    6700 7500
+	-1   0    0    1
+$EndComp
+Wire Wire Line
+	6700 7500 6700 7250
+Text Label 6700 7350 0    50   ~ 0
+BATT
+Wire Wire Line
+	3000 2650 3600 2650
+Wire Wire Line
+	3000 2750 3600 2750
+Text Label 3150 2650 0    50   ~ 0
+INT1
+Text Label 3150 2750 0    50   ~ 0
+INT2
+NoConn ~ 4050 6100
+NoConn ~ 3000 3650
+NoConn ~ 3000 3750
+NoConn ~ 3000 3850
+NoConn ~ 3000 3950
+NoConn ~ 3000 3250
+NoConn ~ 3000 3050
+NoConn ~ 3000 2850
+NoConn ~ 3000 1350
+NoConn ~ 3000 1250
+NoConn ~ 1300 1250
+NoConn ~ 1300 1350
+NoConn ~ 1300 1450
+NoConn ~ 1300 1550
+NoConn ~ 1300 1650
+NoConn ~ 1300 1850
+NoConn ~ 1300 1950
+NoConn ~ 1300 2050
+NoConn ~ 1300 2150
+NoConn ~ 1300 2250
+NoConn ~ 1300 2350
+NoConn ~ 1300 2950
+NoConn ~ 1300 3050
+NoConn ~ 1300 4050
+NoConn ~ 6800 3300
+NoConn ~ 5300 3600
+NoConn ~ 600  4100
+$Comp
+L Device:C_Small C13
+U 1 1 5EFB086A
+P 4450 4800
+F 0 "C13" H 4542 4846 50  0000 L CNN
+F 1 "4.7uF" H 4542 4755 50  0000 L CNN
+F 2 "Capacitors_SMD:C_0603_HandSoldering" H 4450 4800 50  0001 C CNN
+F 3 "~" H 4450 4800 50  0001 C CNN
+	1    4450 4800
+	1    0    0    -1
+$EndComp
+Connection ~ 4450 4700
+Wire Wire Line
+	4450 4700 4550 4700
+$Comp
+L nrf-rescue:(GND)-power1 #PWR0101
+U 1 1 5EFB1BFF
+P 4450 4900
+AR Path="/5EFB1BFF" Ref="#PWR0101"  Part="1"
+AR Path="/5C2799D2/5EFB1BFF" Ref="#PWR?"  Part="1"
+AR Path="/5D08BD3C/5EFB1BFF" Ref="#PWR?"  Part="1"
+F 0 "#PWR0101" H 4450 4900 30  0001 C CNN
+F 1 "(GND)" H 4450 4900 30  0001 C CNN
+F 2 "" H 4450 4900 60  0000 C CNN
+F 3 "" H 4450 4900 60  0000 C CNN
+	1    4450 4900
+	1    0    0    -1
+$EndComp
 $EndSCHEMATC

Commit message: Layout board
Parts:
- removed D2: GREEN, LEDs:LED_0805, symbol Device:LED
- removed R5: 1K, Resistors_SMD:R_0603_HandSoldering, symbol Device:R
Connections:
- net labels added: PWR_CHRGING
- net labels removed: PWR_SENSE, PWR_STAT
- wire segments 271 -> 262
- no-connect marks 27 -> 29
Changed lines of the file:
@@
 EESchema Schematic File Version 4
-LIBS:nrf-cache
-EELAYER 29 0
+EELAYER 30 0
 EELAYER END
 $Descr USLegal 14000 8500
@@
 Wire Wire Line
 	11950 5950 11950 6150
-Wire Wire Line
-	12550 5250 12950 5250
 Text Label 10900 5250 0    50   ~ 0
 QSPI_DATA0
@@
 Text Label 10900 5650 0    50   ~ 0
 QSPI_DATA3
-Text Label 12500 5250 0    50   ~ 0
-QSPI_DATA1
 $Comp
 L power:(GND) #PWR022
@@
 Wire Wire Line
 	1300 3150 1000 3150
-Text Label 1050 3150 0    50   ~ 0
-BTN_1
-Wire Wire Line
-	1300 3250 1000 3250
-Wire Wire Line
-	1300 3350 1000 3350
 Wire Wire Line
 	1300 3450 1000 3450
-Text Label 1050 3250 0    50   ~ 0
-BTN_2
-Text Label 1050 3350 0    50   ~ 0
-BTN_3
 Text Label 1050 3450 0    50   ~ 0
 BTN_4
@@
 	10900 4200 10900 4250
 Connection ~ 10900 4200
-Wire Wire Line
-	850  2550 1300 2550
-Text Label 900  2550 0    50   ~ 0
-LIGHT1
-Wire Wire Line
-	1300 2850 850  2850
-Text Label 900  2850 0    50   ~ 0
-LIGHT2
-Wire Wire Line
-	1300 1750 850  1750
-Text Label 900  1750 0    50   ~ 0
-LIGHT3
 Wire Wire Line
 	3000 1550 3600 1550
@@
 	2050 4650 2050 4600
 $Comp
-L Device:R R5
-U 1 1 5EC59AD5
-P 1600 5200
-AR Path="/5EC59AD5" Ref="R5"  Part="1"
-AR Path="/5C2799D2/5EC59AD5" Ref="R?"  Part="1"
-AR Path="/5D08BD3C/5EC59AD5" Ref="R?"  Part="1"
-F 0 "R5" V 1680 5200 50  0000 C CNN
-F 1 "1K" V 1600 5200 50  0000 C CNN
-F 2 "Resistors_SMD:R_0603_HandSoldering" V 1530 5200 50  0001 C CNN
-F 3 "" H 1600 5200 50  0000 C CNN
-	1    1600 5200
-	1    0    0    -1
-$EndComp
-$Comp
 L Device:R R4
 U 1 1 5EC59ADB
@@
 $EndComp
 Wire Wire Line
-	2850 5400 2350 5400
-Wire Wire Line
-	2350 5400 2350 5650
-Wire Wire Line
-	2350 5650 1600 5650
-Wire Wire Line
-	1600 5650 1600 5450
-Wire Wire Line
 	2850 5500 2450 5500
 Wire Wire Line
 	2450 5500 2450 5750
-$Comp
-L Device:LED D2
-U 1 1 5EC59AE7
-P 1600 4800
-AR Path="/5EC59AE7" Ref="D2"  Part="1"
-AR Path="/5C2799D2/5EC59AE7" Ref="D?"  Part="1"
-AR Path="/5D08BD3C/5EC59AE7" Ref="D?"  Part="1"
-F 0 "D2" H 1600 4900 50  0000 C CNN
-F 1 "GREEN" H 1600 4700 50  0000 C CNN
-F 2 "LEDs:LED_0805" H 1600 4800 50  0001 C CNN
-F 3 "" H 1600 4800 50  0000 C CNN
-	1    1600 4800
-	0    -1   -1   0
-$EndComp
 $Comp
 L Device:LED D1
@@
 $EndComp
 Wire Wire Line
-	1600 4600 1600 4650
-Wire Wire Line
 	1150 4600 1150 4650
 Wire Wire Line
 	1150 4950 1150 5050
-Wire Wire Line
-	1600 4950 1600 5050
 Wire Wire Line
 	1150 5350 1150 5750
@@
 Wire Wire Line
 	4150 6000 4150 6200
-Wire Wire Line
-	1200 5450 1600 5450
-Connection ~ 1600 5450
-Wire Wire Line
-	1600 5450 1600 5350
 Connection ~ 1150 5750
 Text Notes 6900 4850 0    50   ~ 0
@@
 $EndComp
 $Comp
-L power:+5 #PWR032
-U 1 1 5ED2EA24
-P 1600 4600
-F 0 "#PWR032" H 1600 4650 30  0001 C CNN
-F 1 "+5" H 1600 4733 50  0000 C CNN
-F 2 "" H 1600 4600 60  0000 C CNN
-F 3 "" H 1600 4600 60  0000 C CNN
-	1    1600 4600
-	1    0    0    -1
-$EndComp
-$Comp
 L power:+5 #PWR033
 U 1 1 5ED2EDEF
@@
 Wire Wire Line
 	650  5750 1150 5750
-Text Label 650  5750 0    50   ~ 0
-PWR_SENSE
-Text Label 1200 5450 0    50   ~ 0
-PWR_STAT
+Text Label 600  5750 0    50   ~ 0
+PWR_CHRGING
 Wire Wire Line
 	3000 3450 3600 3450
-Wire Wire Line
-	3000 3550 3600 3550
-Text Label 3150 3450 0    50   ~ 0
-PWR_SENSE
-Text Label 3150 3550 0    50   ~ 0
-PWR_STAT
 $Comp
 L Switch:SW_DPST_x2 SW5
@@
 NoConn ~ 3000 1250
 NoConn ~ 1300 1250
-NoConn ~ 1300 1350
-NoConn ~ 1300 1450
 NoConn ~ 1300 1550
 NoConn ~ 1300 1650
@@
 NoConn ~ 1300 1950
 NoConn ~ 1300 2050
-NoConn ~ 1300 2150
 NoConn ~ 1300 2250
-NoConn ~ 1300 2350
-NoConn ~ 1300 2950
 NoConn ~ 1300 3050
 NoConn ~ 1300 4050
@@
 	1    0    0    -1
 $EndComp
+Wire Wire Line
+	1300 1350 850  1350
+Text Label 900  1350 0    50   ~ 0
+LIGHT2
+NoConn ~ 1300 2550
+NoConn ~ 1300 2850
+Wire Wire Line
+	1300 2350 850  2350
+NoConn ~ 1300 1450
+Text Label 900  2350 0    50   ~ 0
+LIGHT1
+Wire Wire Line
+	1300 2150 850  2150
+NoConn ~ 1300 1750
+Text Label 900  2150 0    50   ~ 0
+LIGHT3
+NoConn ~ 2850 5400
+NoConn ~ 2850 5200
+Text Label 3150 3450 0    50   ~ 0
+PWR_CHRGING
+Wire Wire Line
+	1300 2950 1000 2950
+Text Label 1050 2950 0    50   ~ 0
+BTN_3
+Text Label 1050 3150 0    50   ~ 0
+BTN_2
+Wire Wire Line
+	1300 3350 1000 3350
+NoConn ~ 1300 3250
+Text Label 1050 3350 0    50   ~ 0
+BTN_1
+Wire Wire Line
+	12550 5250 13100 5250
+Text Label 12650 5250 0    50   ~ 0
+QSPI_DATA1
 $EndSCHEMATC

Commit message: Layout board
Parts:
- removed D1: ORANGE, LEDs:LED_0805, symbol Device:LED
- added TP5: TestPoint, Measurement_Points:Measurement_Point_Square-SMD-Pad_Small, symbol Connector:TestPoint
- R4: value 1K -> 10K
Connections:
- no-connect marks 29 -> 30
Changed lines of the file:
@@
 AR Path="/5D08BD3C/5EC59ADB" Ref="R?"  Part="1"
 F 0 "R4" V 1230 5200 50  0000 C CNN
-F 1 "1K" V 1150 5200 50  0000 C CNN
+F 1 "10K" V 1150 5200 50  0000 C CNN
 F 2 "Resistors_SMD:R_0603_HandSoldering" V 1080 5200 50  0001 C CNN
 F 3 "" H 1150 5200 50  0000 C CNN
@@
 Wire Wire Line
 	2450 5500 2450 5750
-$Comp
-L Device:LED D1
-U 1 1 5EC59AED
-P 1150 4800
-AR Path="/5EC59AED" Ref="D1"  Part="1"
-AR Path="/5C2799D2/5EC59AED" Ref="D?"  Part="1"
-AR Path="/5D08BD3C/5EC59AED" Ref="D?"  Part="1"
-F 0 "D1" H 1150 4900 50  0000 C CNN
-F 1 "ORANGE" H 1150 4700 50  0000 C CNN
-F 2 "LEDs:LED_0805" H 1150 4800 50  0001 C CNN
-F 3 "" H 1150 4800 50  0000 C CNN
-	1    1150 4800
-	0    -1   -1   0
-$EndComp
-Wire Wire Line
-	1150 4600 1150 4650
 Wire Wire Line
 	1150 4950 1150 5050
@@
 L power:+5 #PWR031
 U 1 1 5ED2E209
-P 1150 4600
-F 0 "#PWR031" H 1150 4650 30  0001 C CNN
-F 1 "+5" H 1150 4733 50  0000 C CNN
-F 2 "" H 1150 4600 60  0000 C CNN
-F 3 "" H 1150 4600 60  0000 C CNN
-	1    1150 4600
+P 1150 4950
+F 0 "#PWR031" H 1150 5000 30  0001 C CNN
+F 1 "+5" H 1150 5083 50  0000 C CNN
+F 2 "" H 1150 4950 60  0000 C CNN
+F 3 "" H 1150 4950 60  0000 C CNN
+	1    1150 4950
 	1    0    0    -1
 $EndComp
@@
 $EndComp
 Wire Wire Line
-	650  5750 1150 5750
-Text Label 600  5750 0    50   ~ 0
+	650  5750 800  5750
+Text Label 700  5750 0    50   ~ 0
 PWR_CHRGING
 Wire Wire Line
@@
 NoConn ~ 6800 3300
 NoConn ~ 5300 3600
-NoConn ~ 600  4100
 $Comp
 L Device:C_Small C13
@@
 NoConn ~ 2850 5400
 NoConn ~ 2850 5200
-Text Label 3150 3450 0    50   ~ 0
+Text Label 3050 3450 0    50   ~ 0
 PWR_CHRGING
 Wire Wire Line
@@
 Text Label 12650 5250 0    50   ~ 0
 QSPI_DATA1
+NoConn ~ 3000 3550
+NoConn ~ 6100 2900
+$Comp
+L Connector:TestPoint TP5
+U 1 1 5ED3684F
+P 800 5750
+F 0 "TP5" H 742 5776 50  0000 R CNN
+F 1 "TestPoint" H 742 5867 50  0000 R CNN
+F 2 "Measurement_Points:Measurement_Point_Square-SMD-Pad_Small" H 1000 5750 50  0001 C CNN
+F 3 "~" H 1000 5750 50  0001 C CNN
+	1    800  5750
+	1    0    0    -1
+$EndComp
+Connection ~ 800  5750
+Wire Wire Line
+	800  5750 1150 5750
 $EndSCHEMATC
