File: nrf.sch (KiCad schematic (older format))
At the start: 55 parts, among them IC1 BMA423, IC2 113990582, J2 Conn_01x05, J7 Conn_01x12, Q1 SI3139K, Q2 MGSF1N02L, Q3 SI3139K, Q4 SI3139K, SW1 UP, SW2 MID, SW3 DOWN, SW4 RESET, SW5 BACK, U1 GD25Q16, U2 C0720B001F, U3 MCP73871-xxI_ML, U4 MIC5219-3.3YM5, X1 32.768

Commit message: Layout board
Parts:
- added J1: Conn_01x10, Pin_Headers:Pin_Header_Straight_1x10_Pitch2.54mm, symbol Connector_Generic:Conn_01x10
- Q1, Q3, Q4: footprint TO_SOT_Packages_SMD:SOT-23 -> TO_SOT_Packages_SMD:SOT-723_Handsoldering
Connections:
- wire segments 262 -> 275
Changed lines of the file:
@@
 QSPI_DATA1
-Wire Wire Line
-	3000 2550 3600 2550
 Wire Wire Line
 	3000 1950 3600 1950
@@
 Wire Wire Line
 	1300 3150 1000 3150
-Wire Wire Line
-	1300 3450 1000 3450
-Text Label 1050 3450 0    50   ~ 0
+Text Label 900  1450 0    50   ~ 0
 BTN_4
 $Comp
@@
 Wire Wire Line
 	1300 3550 800  3550
-Text Label 850  3550 0    50   ~ 0
+Text Label 3150 2750 0    50   ~ 0
 MOTOR_PWM
 $Comp
@@
 Text Label 3150 2250 0    50   ~ 0
 QSPI_CS
-Text Label 3150 2350 0    50   ~ 0
+Text Label 3150 2650 0    50   ~ 0
 QSPI_DATA2
-Wire Wire Line
-	1300 3850 1000 3850
-Text Label 1050 3850 0    50   ~ 0
+Text Label 3150 1250 0    50   ~ 0
 SDA
-Wire Wire Line
-	1300 3650 1000 3650
-Text Label 1050 3650 0    50   ~ 0
+Text Label 3150 1350 0    50   ~ 0
 SCL
 $Comp
@@
 F 0 "Q1" V 10943 3250 50  0000 C CNN
 F 1 "SI3139K" V 10852 3250 50  0000 C CNN
-F 2 "TO_SOT_Packages_SMD:SOT-23" H 10800 3175 50  0001 L CIN
+F 2 "TO_SOT_Packages_SMD:SOT-723_Handsoldering" H 10800 3175 50  0001 L CIN
 F 3 "http://www.vishay.com/docs/70209/70209.pdf" H 10600 3250 50  0001 L CNN
 	1    10600 3250
@@
 F 0 "Q3" V 12593 3250 50  0000 C CNN
 F 1 "SI3139K" V 12502 3250 50  0000 C CNN
-F 2 "TO_SOT_Packages_SMD:SOT-23" H 12450 3175 50  0001 L CIN
+F 2 "TO_SOT_Packages_SMD:SOT-723_Handsoldering" H 12450 3175 50  0001 L CIN
 F 3 "http://www.vishay.com/docs/70209/70209.pdf" H 12250 3250 50  0001 L CNN
 	1    12250 3250
@@
 F 0 "Q4" V 12593 4000 50  0000 C CNN
 F 1 "SI3139K" V 12502 4000 50  0000 C CNN
-F 2 "TO_SOT_Packages_SMD:SOT-23" H 12450 3925 50  0001 L CIN
+F 2 "TO_SOT_Packages_SMD:SOT-723_Handsoldering" H 12450 3925 50  0001 L CIN
 F 3 "http://www.vishay.com/docs/70209/70209.pdf" H 12250 4000 50  0001 L CNN
 	1    12250 4000
@@
 	10900 4200 10900 4250
 Connection ~ 10900 4200
-Wire Wire Line
-	3000 1550 3600 1550
-Text Label 3150 1550 0    50   ~ 0
+Text Label 900  1350 0    50   ~ 0
 SPI_MOSI
-Wire Wire Line
-	3000 1450 3600 1450
-Text Label 3150 1450 0    50   ~ 0
+Text Label 900  1550 0    50   ~ 0
 SPI_SCK
-Wire Wire Line
-	3000 1650 3600 1650
-Text Label 3150 1650 0    50   ~ 0
+Text Label 900  1750 0    50   ~ 0
 SPI_CS
-Wire Wire Line
-	3000 1750 3600 1750
-Text Label 3150 1750 0    50   ~ 0
+Text Label 900  1950 0    50   ~ 0
 SPI_DC
-Text Label 3150 2550 0    50   ~ 0
+Text Label 900  1250 0    50   ~ 0
 SPI_RESET
 $Comp
@@
 Wire Wire Line
 	3000 2750 3600 2750
-Text Label 3150 2650 0    50   ~ 0
+Text Label 1000 4050 0    50   ~ 0
 INT1
-Text Label 3150 2750 0    50   ~ 0
+Text Label 1000 3550 0    50   ~ 0
 INT2
 NoConn ~ 4050 6100
@@
 NoConn ~ 3000 3050
 NoConn ~ 3000 2850
-NoConn ~ 3000 1350
-NoConn ~ 3000 1250
 NoConn ~ 1300 1250
-NoConn ~ 1300 1550
 NoConn ~ 1300 1650
 NoConn ~ 1300 1850
-NoConn ~ 1300 1950
 NoConn ~ 1300 2050
-NoConn ~ 1300 2250
 NoConn ~ 1300 3050
-NoConn ~ 1300 4050
 NoConn ~ 6800 3300
 NoConn ~ 5300 3600
@@
 	1    0    0    -1
 $EndComp
-Wire Wire Line
-	1300 1350 850  1350
-Text Label 900  1350 0    50   ~ 0
+Text Label 900  2250 0    50   ~ 0
 LIGHT2
 NoConn ~ 1300 2550
@@
 Wire Wire Line
 	1300 2350 850  2350
-NoConn ~ 1300 1450
 Text Label 900  2350 0    50   ~ 0
 LIGHT1
 Wire Wire Line
 	1300 2150 850  2150
-NoConn ~ 1300 1750
 Text Label 900  2150 0    50   ~ 0
 LIGHT3
@@
 Wire Wire Line
 	800  5750 1150 5750
+$Comp
+L Connector_Generic:Conn_01x10 J1
+U 1 1 5EF97A2E
+P 9500 1650
+F 0 "J1" H 9580 1692 50  0000 L CNN
+F 1 "Conn_01x10" H 9580 1601 50  0000 L CNN
+F 2 "Pin_Headers:Pin_Header_Straight_1x10_Pitch2.54mm" H 9500 1650 50  0001 C CNN
+F 3 "~" H 9500 1650 50  0001 C CNN
+	1    9500 1650
+	1    0    0    -1
+$EndComp
+$Comp
+L power:(GND) #PWR0102
+U 1 1 5EF99340
+P 8800 2350
+F 0 "#PWR0102" H 8800 2350 30  0001 C CNN
+F 1 "(GND)" H 8800 2350 30  0001 C CNN
+F 2 "" H 8800 2350 60  0000 C CNN
+F 3 "" H 8800 2350 60  0000 C CNN
+	1    8800 2350
+	1    0    0    -1
+$EndComp
+Wire Wire Line
+	9300 2150 8800 2150
+Wire Wire Line
+	8800 2150 8800 2350
+$Comp
+L power:+3.3 #PWR?
+U 1 1 5EFAEB0C
+P 8550 850
+AR Path="/5D059B17/5EFAEB0C" Ref="#PWR?"  Part="1"
+AR Path="/5EFAEB0C" Ref="#PWR0103"  Part="1"
+F 0 "#PWR0103" H 8550 900 30  0001 C CNN
+F 1 "+3.3" H 8550 983 50  0000 C CNN
+F 2 "" H 8550 850 60  0000 C CNN
+F 3 "" H 8550 850 60  0000 C CNN
+	1    8550 850
+	1    0    0    -1
+$EndComp
+Wire Wire Line
+	9300 1250 8800 1250
+Wire Wire Line
+	9300 1350 8800 1350
+Wire Wire Line
+	9300 1450 8800 1450
+Wire Wire Line
+	9300 1550 8800 1550
+Wire Wire Line
+	9300 1650 8800 1650
+Wire Wire Line
+	9300 1750 8800 1750
+Wire Wire Line
+	9300 1850 8800 1850
+Wire Wire Line
+	9300 1950 8800 1950
+Text Label 8850 1250 0    50   ~ 0
+LIGHT1
+Text Label 8850 1350 0    50   ~ 0
+LIGHT2
+Text Label 8850 1450 0    50   ~ 0
+LIGHT3
+Text Label 8850 1950 0    50   ~ 0
+SPI_RESET
+Text Label 8850 1850 0    50   ~ 0
+SPI_MOSI
+Text Label 8850 1750 0    50   ~ 0
+SPI_SCK
+Text Label 8850 1650 0    50   ~ 0
+SPI_CS
+Text Label 8850 1550 0    50   ~ 0
+SPI_DC
+Wire Wire Line
+	8550 850  8550 2050
+Wire Wire Line
+	8550 2050 9300 2050
+Wire Wire Line
+	1300 1950 850  1950
+Wire Wire Line
+	1300 1250 850  1250
+NoConn ~ 3000 2550
+Wire Wire Line
+	1300 1350 850  1350
+Wire Wire Line
+	1300 1550 850  1550
+NoConn ~ 3000 1450
+Wire Wire Line
+	1300 1750 850  1750
+Wire Wire Line
+	1300 2250 850  2250
+NoConn ~ 3000 1550
+NoConn ~ 3000 1650
+NoConn ~ 3000 1750
+Wire Wire Line
+	1300 1450 850  1450
+NoConn ~ 1300 3450
+Wire Wire Line
+	3000 1350 3600 1350
+Wire Wire Line
+	3000 1250 3600 1250
+NoConn ~ 1300 3650
+NoConn ~ 1300 3850
+Wire Wire Line
+	1300 4050 850  4050
 $EndSCHEMATC

Commit message: More layout changes
Parts:
- removed TP5: TestPoint, Measurement_Points:Measurement_Point_Square-SMD-Pad_Small, symbol Connector:TestPoint
- added C14: ??pF, Capacitors_SMD:C_0603_HandSoldering, symbol Device:C_Small
- added J3: Conn_01x05, Pin_Headers:Pin_Header_Straight_1x05_Pitch2.54mm, symbol Connector_Generic:Conn_01x05
- added R5: 1, Resistors_SMD:R_0603_HandSoldering, symbol Device:R
Connections:
- net labels added: LEDA
- wire segments 275 -> 289
- no-connect marks 30 -> 26
Other:
- note added: "Digital Accel Sensor"
- moved on the sheet: J2
Changed lines of the file:
@@
 $EndComp
 Wire Wire Line
-	6950 1150 6850 1150
+	6550 1150 6850 1150
 Wire Wire Line
 	6850 1150 6850 1000
 Wire Wire Line
-	6950 1550 6850 1550
+	6550 1550 6850 1550
 Wire Wire Line
 	6850 1550 6850 1800
@@
 Text Label 5600 2300 0    50   ~ 0
 BTN_4
-$Comp
-L SamacSys_Parts:113990582 IC2
-U 1 1 5EB39C74
-P 1300 1050
-F 0 "IC2" H 2150 1315 50  0000 C CNN
-F 1 "113990582" H 2150 1224 50  0000 C CNN
-F 2 "SamacSys_Parts:113990582" H 2850 1150 50  0001 L CNN
-F 3 "http://www.raytac.com/download/index.php?index_id=24" H 2850 1050 50  0001 L CNN
-F 4 "Bluetooth Modules (802.15.1) MDBT50Q-1M nRF52840 Based BLE Module" H 2850 950 50  0001 L CNN "Description"
-F 5 "2" H 2850 850 50  0001 L CNN "Height"
-F 6 "713-113990582" H 2850 750 50  0001 L CNN "Mouser Part Number"
-F 7 "https://www.mouser.co.uk/ProductDetail/Seeed-Studio/113990582?qs=0lSvoLzn4L96en1uEjxsrg%3D%3D" H 2850 650 50  0001 L CNN "Mouser Price/Stock"
-F 8 "Seeed Studio" H 2850 550 50  0001 L CNN "Manufacturer_Name"
-F 9 "113990582" H 2850 450 50  0001 L CNN "Manufacturer_Part_Number"
-	1    1300 1050
-	1    0    0    -1
-$EndComp
 $Comp
 L power:(GND) #PWR010
@@
 Text Label 3150 1950 0    50   ~ 0
 QSPI_DATA0
-Wire Wire Line
-	3000 2350 3600 2350
 Wire Wire Line
 	3000 2050 3600 2050
@@
 L Connector_Generic:Conn_01x05 J2
 U 1 1 5D0EA690
-P 7150 1350
-F 0 "J2" H 7230 1392 50  0000 L CNN
-F 1 "Conn_01x05" H 7230 1301 50  0000 L CNN
-F 2 "Pin_Headers:Pin_Header_Straight_1x05_Pitch1.27mm" H 7150 1350 50  0001 C CNN
-F 3 "~" H 7150 1350 50  0001 C CNN
-	1    7150 1350
-	1    0    0    -1
+P 6350 1350
+F 0 "J2" H 6430 1392 50  0000 L CNN
+F 1 "Conn_01x05" H 6430 1301 50  0000 L CNN
+F 2 "Pin_Headers:Pin_Header_Straight_1x05_Pitch1.27mm" H 6350 1350 50  0001 C CNN
+F 3 "~" H 6350 1350 50  0001 C CNN
+	1    6350 1350
+	-1   0    0    1
 $EndComp
 $Comp
@@
 Wire Wire Line
 	1300 3150 1000 3150
-Text Label 900  1450 0    50   ~ 0
+Text Label 3150 2750 0    50   ~ 0
 BTN_4
 $Comp
@@
 Wire Wire Line
 	1300 3550 800  3550
-Text Label 3150 2750 0    50   ~ 0
+Text Label 850  3850 0    50   ~ 0
 MOTOR_PWM
 $Comp
@@
 	10350 1850 11000 1850
 Wire Wire Line
-	11000 1850 11000 2250
+	11000 1850 11000 2150
 Connection ~ 11000 2250
 Wire Wire Line
@@
 	11000 1750 11000 1850
 Connection ~ 11000 1850
-Wire Wire Line
-	10350 2050 11150 2050
 Wire Wire Line
 	11150 2050 11150 1950
@@
 $EndComp
 Wire Wire Line
-	10350 2150 10800 2150
-Text Label 10550 2150 0    50   ~ 0
-LEDK
-Wire Wire Line
 	10350 1950 11150 1950
 Connection ~ 11150 1950
@@
 SPI_RESET
 Wire Wire Line
-	10350 1150 11100 1150
-Wire Wire Line
-	11100 1150 11100 1300
+	10350 1150 11350 1150
+Wire Wire Line
+	11350 1150 11350 1300
 $Comp
 L power:(GND) #PWR026
 U 1 1 5EC295E8
-P 11100 1300
-F 0 "#PWR026" H 11100 1300 30  0001 C CNN
-F 1 "(GND)" H 11100 1300 30  0001 C CNN
-F 2 "" H 11100 1300 60  0000 C CNN
-F 3 "" H 11100 1300 60  0000 C CNN
-	1    11100 1300
+P 11350 1300
+F 0 "#PWR026" H 11350 1300 30  0001 C CNN
+F 1 "(GND)" H 11350 1300 30  0001 C CNN
+F 2 "" H 11350 1300 60  0000 C CNN
+F 3 "" H 11350 1300 60  0000 C CNN
+	1    11350 1300
 	1    0    0    -1
 $EndComp
@@
 Text Label 3150 2650 0    50   ~ 0
 QSPI_DATA2
-Text Label 3150 1250 0    50   ~ 0
+Text Label 1050 2850 0    50   ~ 0
 SDA
-Text Label 3150 1350 0    50   ~ 0
+Text Label 1050 3050 0    50   ~ 0
 SCL
 $Comp
@@
 	1    0    0    -1
 $EndComp
-Connection ~ 11150 2050
 Wire Wire Line
 	11150 2250 11000 2250
@@
 	11150 3150 11350 3150
 Text Label 11150 3150 0    50   ~ 0
-LEDK
+LEDA
 $Comp
 L power:+3.3 #PWR?
@@
 	12800 3150 13000 3150
 Text Label 12800 3150 0    50   ~ 0
-LEDK
+LEDA
 $Comp
 L power:+3.3 #PWR?
@@
 	12800 3900 13000 3900
 Text Label 12800 3900 0    50   ~ 0
-LEDK
+LEDA
 $Comp
 L Device:C_Small C11
@@
 	1    0    0    -1
 $EndComp
-Wire Wire Line
-	650  5750 800  5750
 Text Label 700  5750 0    50   ~ 0
 PWR_CHRGING
@@
 NoConn ~ 1300 1850
 NoConn ~ 1300 2050
-NoConn ~ 1300 3050
 NoConn ~ 6800 3300
 NoConn ~ 5300 3600
@@
 Text Label 900  2250 0    50   ~ 0
 LIGHT2
-NoConn ~ 1300 2550
-NoConn ~ 1300 2850
 Wire Wire Line
 	1300 2350 850  2350
@@
 NoConn ~ 2850 5400
 NoConn ~ 2850 5200
-Text Label 3050 3450 0    50   ~ 0
+Text Label 3100 1750 0    50   ~ 0
 PWR_CHRGING
 Wire Wire Line
 	1300 2950 1000 2950
-Text Label 1050 2950 0    50   ~ 0
+Text Label 1050 3350 0    50   ~ 0
 BTN_3
 Text Label 1050 3150 0    50   ~ 0
@@
 	1300 3350 1000 3350
 NoConn ~ 1300 3250
-Text Label 1050 3350 0    50   ~ 0
+Text Label 1050 2950 0    50   ~ 0
 BTN_1
 Wire Wire Line
@@
 NoConn ~ 3000 3550
 NoConn ~ 6100 2900
-$Comp
-L Connector:TestPoint TP5
-U 1 1 5ED3684F
-P 800 5750
-F 0 "TP5" H 742 5776 50  0000 R CNN
-F 1 "TestPoint" H 742 5867 50  0000 R CNN
-F 2 "Measurement_Points:Measurement_Point_Square-SMD-Pad_Small" H 1000 5750 50  0001 C CNN
-F 3 "~" H 1000 5750 50  0001 C CNN
-	1    800  5750
-	1    0    0    -1
-$EndComp
-Connection ~ 800  5750
-Wire Wire Line
-	800  5750 1150 5750
 $Comp
 L Connector_Generic:Conn_01x10 J1
@@
 NoConn ~ 3000 1550
 NoConn ~ 3000 1650
-NoConn ~ 3000 1750
 Wire Wire Line
 	1300 1450 850  1450
@@
 	3000 1250 3600 1250
 NoConn ~ 1300 3650
-NoConn ~ 1300 3850
 Wire Wire Line
 	1300 4050 850  4050
+Wire Wire Line
+	1300 2550 850  2550
+NoConn ~ 3000 2350
+Wire Wire Line
+	3000 1750 3600 1750
+Wire Wire Line
+	650  5750 1150 5750
+$Comp
+L Device:R R5
+U 1 1 5F6C25E5
+P 10600 2150
+F 0 "R5" V 10550 2050 50  0000 R CNN
+F 1 "1" V 10600 2250 50  0000 R CNN
+F 2 "Resistors_SMD:R_0603_HandSoldering" V 10530 2150 50  0001 C CNN
+F 3 "~" H 10600 2150 50  0001 C CNN
+	1    10600 2150
+	0    1    1    0
+$EndComp
+Text Label 10750 2150 0    50   ~ 0
+LEDK
+Wire Wire Line
+	10350 2150 10450 2150
+Wire Wire Line
+	10750 2150 11000 2150
+Connection ~ 11000 2150
+Wire Wire Line
+	11000 2150 11000 2250
+Text Label 10550 2050 0    50   ~ 0
+LEDA
+Wire Wire Line
+	10350 2050 10750 2050
+$Comp
+L Device:C_Small C14
+U 1 1 5F738E71
+P 8000 7400
+AR Path="/5F738E71" Ref="C14"  Part="1"
+AR Path="/5C2799D2/5F738E71" Ref="C?"  Part="1"
+AR Path="/5D08445F/5F738E71" Ref="C?"  Part="1"
+AR Path="/5D08BD3C/5F738E71" Ref="C?"  Part="1"
+F 0 "C14" H 8100 7400 50  0000 L CNN
+F 1 "??pF" H 7950 7500 50  0000 L CNN
+F 2 "Capacitors_SMD:C_0603_HandSoldering" H 8000 7400 50  0001 C CNN
+F 3 "" H 8000 7400 50  0000 C CNN
+	1    8000 7400
+	1    0    0    -1
+$EndComp
+$Comp
+L nrf-rescue:(GND)-power1 #PWR032
+U 1 1 5F7394B3
+P 8000 7650
+AR Path="/5F7394B3" Ref="#PWR032"  Part="1"
+AR Path="/5C2799D2/5F7394B3" Ref="#PWR?"  Part="1"
+AR Path="/5D08BD3C/5F7394B3" Ref="#PWR?"  Part="1"
+F 0 "#PWR032" H 8000 7650 30  0001 C CNN
+F 1 "(GND)" H 8000 7650 30  0001 C CNN
+F 2 "" H 8000 7650 60  0000 C CNN
+F 3 "" H 8000 7650 60  0000 C CNN
+	1    8000 7650
+	1    0    0    -1
+$EndComp
+Wire Wire Line
+	8000 7500 8000 7650
+Wire Wire Line
+	8000 7300 8000 7050
+Text Label 8000 7250 1    50   ~ 0
+SPI_MOSI
+$Comp
+L Connector_Generic:Conn_01x05 J3
+U 1 1 5F7A4F6A
+P 6400 6500
+F 0 "J3" H 6480 6542 50  0000 L CNN
+F 1 "Conn_01x05" H 6480 6451 50  0000 L CNN
+F 2 "Pin_Headers:Pin_Header_Straight_1x05_Pitch2.54mm" H 6400 6500 50  0001 C CNN
+F 3 "~" H 6400 6500 50  0001 C CNN
+	1    6400 6500
+	-1   0    0    1
+$EndComp
+Wire Wire Line
+	6600 6500 7300 6500
+Text Label 6750 6500 0    50   ~ 0
+PWR_CHRGING
+$Comp
+L nrf-rescue:(GND)-power1 #PWR051
+U 1 1 5F7D59F0
+P 6800 6900
+AR Path="/5F7D59F0" Ref="#PWR051"  Part="1"
+AR Path="/5C2799D2/5F7D59F0" Ref="#PWR?"  Part="1"
+AR Path="/5D08BD3C/5F7D59F0" Ref="#PWR?"  Part="1"
+F 0 "#PWR051" H 6800 6900 30  0001 C CNN
+F 1 "(GND)" H 6800 6900 30  0001 C CNN
+F 2 "" H 6800 6900 60  0000 C CNN
+F 3 "" H 6800 6900 60  0000 C CNN
+	1    6800 6900
+	1    0    0    -1
+$EndComp
+Wire Wire Line
+	6600 6700 6800 6700
+Wire Wire Line
+	6800 6700 6800 6900
+Wire Wire Line
+	6600 6300 6800 6300
+Wire Wire Line
+	6800 6300 6800 6100
+$Comp
+L power:+5 #PWR050
+U 1 1 5F804326
+P 6800 6100
+F 0 "#PWR050" H 6800 6150 30  0001 C CNN
+F 1 "+5" H 6800 6233 50  0000 C CNN
+F 2 "" H 6800 6100 60  0000 C CNN
+F 3 "" H 6800 6100 60  0000 C CNN
+	1    6800 6100
+	1    0    0    -1
+$EndComp
+$Comp
+L power:+3.3 #PWR?
+U 1 1 5F87C00F
+P 7500 6100
+AR Path="/5D09E285/5F87C00F" Ref="#PWR?"  Part="1"
+AR Path="/5F87C00F" Ref="#PWR0104"  Part="1"
+F 0 "#PWR0104" H 7500 6150 30  0001 C CNN
+F 1 "+3.3" H 7500 6233 50  0000 C CNN
+F 2 "" H 7500 6100 60  0000 C CNN
+F 3 "" H 7500 6100 60  0000 C CNN
+	1    7500 6100
+	1    0    0    -1
+$EndComp
+Wire Wire Line
+	7500 6600 7500 6100
+Wire Wire Line
+	6600 6600 7500 6600
+Text Notes 6250 2650 0    50   ~ 0
+Digital Accel Sensor
+$Comp
+L SamacSys_Parts:113990582 IC2
+U 1 1 5EB39C74
+P 1300 1050
+F 0 "IC2" H 2150 1315 50  0000 C CNN
+F 1 "113990582" H 2150 1224 50  0000 C CNN
+F 2 "SamacSys_Parts:113990582" H 2850 1150 50  0001 L CNN
+F 3 "http://www.raytac.com/download/index.php?index_id=24" H 2850 1050 50  0001 L CNN
+F 4 "Bluetooth Modules (802.15.1) MDBT50Q-1M nRF52840 Based BLE Module" H 2850 950 50  0001 L CNN "Description"
+F 5 "2" H 2850 850 50  0001 L CNN "Height"
+F 6 "713-113990582" H 2850 750 50  0001 L CNN "Mouser Part Number"
+F 7 "https://www.mouser.co.uk/ProductDetail/Seeed-Studio/113990582?qs=0lSvoLzn4L96en1uEjxsrg%3D%3D" H 2850 650 50  0001 L CNN "Mouser Price/Stock"
+F 8 "Seeed Studio" H 2850 550 50  0001 L CNN "Manufacturer_Name"
+F 9 "113990582" H 2850 450 50  0001 L CNN "Manufacturer_Part_Number"
+	1    1300 1050
+	1    0    0    -1
+$EndComp
+Wire Wire Line
+	1300 3850 800  3850
+Wire Wire Line
+	1300 3050 1000 3050
+Wire Wire Line
+	1300 2850 1000 2850
 $EndSCHEMATC

Commit message: Board Update
Parts:
- removed R18, R19: 10K, Resistors_SMD:R_0603_HandSoldering, symbol Device:R_Small
- removed SW4: RESET, Buttons_Switches_SMD:SW_SPST_B3U-1000P, symbol Switch:SW_DPST_x2
- added L1: 10uH, Inductor_SMD:L_0603_1608Metric_Pad1.05x0.95mm_HandSolder, symbol Device:L
- added R20, R21: 1M, Resistor_SMD:R_0201_0603Metric_Pad0.64x0.40mm_HandSolder, symbol Device:R_Small
- C1, C10, C11, C12, C13, C14, C2, C3, C4, C5, C6, C8: footprint Capacitors_SMD:C_0603_HandSoldering -> Capacitor_SMD:C_0201_0603Metric_Pad0.64x0.40mm_HandSolder
- C7: value 470pF -> 0.1uF; footprint Capacitors_SMD:C_0603_HandSoldering -> Capacitor_SMD:C_0201_0603Metric_Pad0.64x0.40mm_HandSolder
- C9: value 470pF -> 4.7uF; footprint Capacitors_SMD:C_0603_HandSoldering -> Capacitor_SMD:C_0201_0603Metric_Pad0.64x0.40mm_HandSolder
- IC2: footprint SamacSys_Parts:113990582 -> RF_Module:Raytac_MDBT50Q; symbol SamacSys_Parts:113990582 -> RF_Module:MDBT50Q-1MV2
- R1, R10, R11, R12, R13, R14, R15, R16, R17, R2, R3, R4, R5, R6, R7, R8, R9: footprint Resistors_SMD:R_0603_HandSoldering -> Resistor_SMD:R_0201_0603Metric_Pad0.64x0.40mm_HandSolder
- TP1, TP2, TP3, TP4: footprint Measurement_Points:Measurement_Point_Square-SMD-Pad_Big -> TestPoint:TestPoint_Pad_2.0x2.0mm
- U3: symbol nrf-rescue:MCP73871-xxI_ML-microchip -> Microchip:MCP73871-xxI_ML
Connections:
- net labels added: BATT_LVL
- wire segments 289 -> 279
- no-connect marks 26 -> 9
Other:
- moved on the sheet: C12, C13, C3, C6, C7, C9, J3, R14, R15, R16, R4, R6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
