File: nrf.sch (KiCad schematic (older format))
At the start: 58 parts, among them IC1 BMA423, IC2 113990582, J1 Conn_01x10, J2 Conn_01x05, J3 Conn_01x05, J7 Conn_01x12, Q1 SI3139K, Q2 MGSF1N02L, Q3 SI3139K, Q4 SI3139K, SW1 UP, SW2 MID, SW3 DOWN, SW5 BACK, U1 GD25Q16, U2 C0720B001F, U3 MCP73871-xxI_ML, U4 MIC5219-3.3YM5, X1 32.768

Commit message: Change resistors to 0603 imperial
Parts:
- C1, C10, C11, C12, C13, C14, C2, C3, C4, C5, C6, C7, C8, C9: footprint Capacitor_SMD:C_0201_0603Metric_Pad0.64x0.40mm_HandSolder -> Capacitor_SMD:C_0603_1608Metric_Pad1.08x0.95mm_HandSolder
- R1, R10, R11, R12, R13, R14, R15, R16, R17, R2, R20, R21, R3, R4, R5, R6, R7, R8, R9: footprint Resistor_SMD:R_0201_0603Metric_Pad0.64x0.40mm_HandSolder -> Resistor_SMD:R_0603_1608Metric_Pad0.98x0.95mm_HandSolder

Commit message: Board Update
Parts:
- added TP5, TP6, TP7: (no value), TestPoint:TestPoint_Pad_D1.0mm, symbol Connector:TestPoint
- Q1, Q3, Q4: footprint TO_SOT_Packages_SMD:SOT-723_Handsoldering -> Package_TO_SOT_SMD:SOT-723
- Q2: footprint TO_SOT_Packages_SMD:SOT-23 -> Package_TO_SOT_SMD:SOT-23
Connections:
- net labels added: MOTOR_3.3, MOTOR_GND
- wire segments 279 -> 282
Changed lines of the file:
@@
 F 0 "Q2" H 12906 1996 50  0000 L CNN
 F 1 "MGSF1N02L" H 12650 2150 50  0000 L CNN
-F 2 "TO_SOT_Packages_SMD:SOT-23" H 12900 1875 50  0001 L CIN
+F 2 "Package_TO_SOT_SMD:SOT-23" H 12900 1875 50  0001 L CIN
 F 3 "https://www.fairchildsemi.com/datasheets/2N/2N7002.pdf" H 12700 1950 50  0001 L CNN
 	1    12700 1950
@@
 F 0 "Q1" V 10943 3250 50  0000 C CNN
 F 1 "SI3139K" V 10852 3250 50  0000 C CNN
-F 2 "TO_SOT_Packages_SMD:SOT-723_Handsoldering" H 10800 3175 50  0001 L CIN
+F 2 "Package_TO_SOT_SMD:SOT-723" H 10800 3175 50  0001 L CIN
 F 3 "http://www.vishay.com/docs/70209/70209.pdf" H 10600 3250 50  0001 L CNN
 	1    10600 3250
@@
 F 0 "Q3" V 12593 3250 50  0000 C CNN
 F 1 "SI3139K" V 12502 3250 50  0000 C CNN
-F 2 "TO_SOT_Packages_SMD:SOT-723_Handsoldering" H 12450 3175 50  0001 L CIN
+F 2 "Package_TO_SOT_SMD:SOT-723" H 12450 3175 50  0001 L CIN
 F 3 "http://www.vishay.com/docs/70209/70209.pdf" H 12250 3250 50  0001 L CNN
 	1    12250 3250
@@
 F 0 "Q4" V 12593 4000 50  0000 C CNN
 F 1 "SI3139K" V 12502 4000 50  0000 C CNN
-F 2 "TO_SOT_Packages_SMD:SOT-723_Handsoldering" H 12450 3925 50  0001 L CIN
+F 2 "Package_TO_SOT_SMD:SOT-723" H 12450 3925 50  0001 L CIN
 F 3 "http://www.vishay.com/docs/70209/70209.pdf" H 12250 4000 50  0001 L CNN
 	1    12250 4000
@@
 Wire Wire Line
 	8000 7300 8000 7050
+$Comp
+L Connector:TestPoint TP6
+U 1 1 5FA7DF75
+P 3750 7550
+F 0 "TP6" H 3808 7668 50  0000 L CNN
+F 1 " " H 3808 7577 50  0000 L CNN
+F 2 "TestPoint:TestPoint_Pad_D1.0mm" H 3950 7550 50  0001 C CNN
+F 3 "~" H 3950 7550 50  0001 C CNN
+	1    3750 7550
+	-1   0    0    1
+$EndComp
+$Comp
+L Connector:TestPoint TP7
+U 1 1 5FA7E25F
+P 4000 7200
+F 0 "TP7" H 4058 7318 50  0000 L CNN
+F 1 " " H 4058 7227 50  0000 L CNN
+F 2 "TestPoint:TestPoint_Pad_D1.0mm" H 4200 7200 50  0001 C CNN
+F 3 "~" H 4200 7200 50  0001 C CNN
+	1    4000 7200
+	1    0    0    -1
+$EndComp
+Text Label 11900 1200 0    50   ~ 0
+MOTOR_3.3
+Text Label 12350 2450 0    50   ~ 0
+MOTOR_GND
+Text Label 3750 7550 1    50   ~ 0
+MOTOR_3.3
+$Comp
+L power:+3.3 #PWR?
+U 1 1 5FA96F62
+P 3750 7100
+AR Path="/5D09E285/5FA96F62" Ref="#PWR?"  Part="1"
+AR Path="/5FA96F62" Ref="#PWR08"  Part="1"
+F 0 "#PWR08" H 3750 7150 30  0001 C CNN
+F 1 "+3.3" H 3750 7233 50  0000 C CNN
+F 2 "" H 3750 7100 60  0000 C CNN
+F 3 "" H 3750 7100 60  0000 C CNN
+	1    3750 7100
+	1    0    0    -1
+$EndComp
+Wire Wire Line
+	3750 7100 3750 7550
+$Comp
+L power:(GND) #PWR?
+U 1 1 5FAB0BDB
+P 4000 7650
+AR Path="/5DA394ED/5FAB0BDB" Ref="#PWR?"  Part="1"
+AR Path="/5FAB0BDB" Ref="#PWR010"  Part="1"
+F 0 "#PWR010" H 4000 7650 30  0001 C CNN
+F 1 "(GND)" H 4000 7650 30  0001 C CNN
+F 2 "" H 4000 7650 60  0000 C CNN
+F 3 "" H 4000 7650 60  0000 C CNN
+	1    4000 7650
+	1    0    0    -1
+$EndComp
+Wire Wire Line
+	4000 7200 4000 7650
+Text Label 4000 7550 1    50   ~ 0
+MOTOR_GND
+$Comp
+L Connector:TestPoint TP5
+U 1 1 5FAFD167
+P 3400 7550
+F 0 "TP5" H 3458 7668 50  0000 L CNN
+F 1 " " H 3458 7577 50  0000 L CNN
+F 2 "TestPoint:TestPoint_Pad_D1.0mm" H 3600 7550 50  0001 C CNN
+F 3 "~" H 3600 7550 50  0001 C CNN
+	1    3400 7550
+	-1   0    0    1
+$EndComp
+Wire Wire Line
+	3400 7550 3400 7050
+Text Label 3400 7550 1    50   ~ 0
+MOTOR_PWM
 $EndSCHEMATC

Commit message: Board Update
Connections:
- no-connect marks 9 -> 7
Changed lines of the file:
@@
 Wire Wire Line
 	3650 4400 3150 4400
-Text Label 3200 4200 0    50   ~ 0
+Text Label 3300 4200 0    50   ~ 0
 MOTOR_PWM
 $Comp
@@
 	10900 4200 10900 4250
 Connection ~ 10900 4200
-Text Label 1150 4300 0    50   ~ 0
+Text Label 1150 4700 0    50   ~ 0
 SPI_MOSI
 Text Label 1150 4500 0    50   ~ 0
 SPI_SCK
-Text Label 1150 4700 0    50   ~ 0
+Text Label 1150 4300 0    50   ~ 0
 SPI_CS
+Text Label 1150 4200 0    50   ~ 0
+SPI_DC
 Text Label 1150 2300 0    50   ~ 0
-SPI_DC
-Text Label 1150 4200 0    50   ~ 0
 SPI_RESET
 $Comp
@@
 Text Label 3300 2300 0    50   ~ 0
 BTN_2
-NoConn ~ 1500 3800
 Text Label 1300 1900 0    50   ~ 0
 BTN_1
@@
 Wire Wire Line
 	1550 2200 1100 2200
-NoConn ~ 1500 4000
 Wire Wire Line
 	3600 4300 3150 4300

Commit message: Update footprints
Parts:
- D4: footprint Diodes_SMD:D_SOD-323 -> Diode_SMD:D_SOD-323_HandSoldering
- IC1: footprint SamacSys_Parts:BMA423 -> Package_LGA_marks:LGA-12_2x2mm_P0.5mm_small_pad
Changed lines of the file:
@@
 F 0 "D4" V 12133 1650 50  0000 C CNN
 F 1 "ZLLS410" V 12224 1650 50  0000 C CNN
-F 2 "Diodes_SMD:D_SOD-323" H 12350 1650 60  0001 C CNN
+F 2 "Diode_SMD:D_SOD-323_HandSoldering" H 12350 1650 60  0001 C CNN
 F 3 "" H 12350 1650 60  0000 C CNN
 	1    12350 1650
@@
 F 0 "IC1" V 6350 2200 50  0000 C CNN
 F 1 "BMA423" V 6200 3200 50  0000 C CNN
-F 2 "SamacSys_Parts:BMA423" H 7050 3400 50  0001 L CNN
+F 2 "Package_LGA_marks:LGA-12_2x2mm_P0.5mm_small_pad" H 7050 3400 50  0001 L CNN
 F 3 "https://componentsearchengine.com/Datasheets/1/BMA423.pdf" H 7050 3300 50  0001 L CNN
 F 4 "Accelerometers Triaxial low-g 12bit Acceleration Sensor" H 7050 3200 50  0001 L CNN "Description"
@@
 NoConn ~ 6200 6400
 NoConn ~ 1550 4600
-NoConn ~ 6800 3300
 NoConn ~ 5300 3600
 $Comp
@@
 Text Label 3400 7550 1    50   ~ 0
 MOTOR_PWM
+NoConn ~ 6800 3300
 $EndSCHEMATC

Commit message: Board updates
Parts:
- removed TP5, TP6, TP7: (no value), TestPoint:TestPoint_Pad_D1.0mm, symbol Connector:TestPoint
- TP1, TP2: footprint TestPoint:TestPoint_Pad_2.0x2.0mm -> TestPoint:TestPoint_Pad_D1.5mm
- U2: footprint my-fp-library:VIBRATION MOTOR COIN 3V FLEX - C0720B001F -> Package_LGA_marks:VIBRATION MOTOR COIN 3V FLEX - C0720B001F
Connections:
- wire segments 282 -> 279
Changed lines of the file:
@@
 F 0 "U2" H 12350 1734 50  0000 C CNN
 F 1 "C0720B001F" H 12350 1643 50  0000 C CNN
-F 2 "my-fp-library:VIBRATION MOTOR COIN 3V FLEX - C0720B001F" H 12350 1300 50  0001 C CNN
+F 2 "Package_LGA_marks:VIBRATION MOTOR COIN 3V FLEX - C0720B001F" H 12350 1300 50  0001 C CNN
 F 3 "http://www.vibration-motor.com/products/download/C0720B001F.pdf" H 12350 1300 50  0001 C CNN
 	1    12350 1300
@@
 F 0 "TP1" H 4442 7576 50  0000 R CNN
 F 1 "TestPoint" H 4442 7667 50  0000 R CNN
-F 2 "TestPoint:TestPoint_Pad_2.0x2.0mm" H 4700 7550 50  0001 C CNN
+F 2 "TestPoint:TestPoint_Pad_D1.5mm" H 4700 7550 50  0001 C CNN
 F 3 "~" H 4700 7550 50  0001 C CNN
 	1    4500 7550
@@
 F 0 "TP2" H 5192 7426 50  0000 R CNN
 F 1 "TestPoint" H 5192 7517 50  0000 R CNN
-F 2 "TestPoint:TestPoint_Pad_2.0x2.0mm" H 5450 7400 50  0001 C CNN
+F 2 "TestPoint:TestPoint_Pad_D1.5mm" H 5450 7400 50  0001 C CNN
 F 3 "~" H 5450 7400 50  0001 C CNN
 	1    5250 7400
@@
 Wire Wire Line
 	8000 7300 8000 7050
-$Comp
-L Connector:TestPoint TP6
-U 1 1 5FA7DF75
-P 3750 7550
-F 0 "TP6" H 3808 7668 50  0000 L CNN
-F 1 " " H 3808 7577 50  0000 L CNN
-F 2 "TestPoint:TestPoint_Pad_D1.0mm" H 3950 7550 50  0001 C CNN
-F 3 "~" H 3950 7550 50  0001 C CNN
-	1    3750 7550
-	-1   0    0    1
-$EndComp
-$Comp
-L Connector:TestPoint TP7
-U 1 1 5FA7E25F
-P 4000 7200
-F 0 "TP7" H 4058 7318 50  0000 L CNN
-F 1 " " H 4058 7227 50  0000 L CNN
-F 2 "TestPoint:TestPoint_Pad_D1.0mm" H 4200 7200 50  0001 C CNN
-F 3 "~" H 4200 7200 50  0001 C CNN
-	1    4000 7200
-	1    0    0    -1
-$EndComp
 Text Label 11900 1200 0    50   ~ 0
 MOTOR_3.3
 Text Label 12350 2450 0    50   ~ 0
 MOTOR_GND
-Text Label 3750 7550 1    50   ~ 0
-MOTOR_3.3
-$Comp
-L power:+3.3 #PWR?
-U 1 1 5FA96F62
-P 3750 7100
-AR Path="/5D09E285/5FA96F62" Ref="#PWR?"  Part="1"
-AR Path="/5FA96F62" Ref="#PWR08"  Part="1"
-F 0 "#PWR08" H 3750 7150 30  0001 C CNN
-F 1 "+3.3" H 3750 7233 50  0000 C CNN
-F 2 "" H 3750 7100 60  0000 C CNN
-F 3 "" H 3750 7100 60  0000 C CNN
-	1    3750 7100
-	1    0    0    -1
-$EndComp
-Wire Wire Line
-	3750 7100 3750 7550
-$Comp
-L power:(GND) #PWR?
-U 1 1 5FAB0BDB
-P 4000 7650
-AR Path="/5DA394ED/5FAB0BDB" Ref="#PWR?"  Part="1"
-AR Path="/5FAB0BDB" Ref="#PWR010"  Part="1"
-F 0 "#PWR010" H 4000 7650 30  0001 C CNN
-F 1 "(GND)" H 4000 7650 30  0001 C CNN
-F 2 "" H 4000 7650 60  0000 C CNN
-F 3 "" H 4000 7650 60  0000 C CNN
-	1    4000 7650
-	1    0    0    -1
-$EndComp
-Wire Wire Line
-	4000 7200 4000 7650
-Text Label 4000 7550 1    50   ~ 0
-MOTOR_GND
-$Comp
-L Connector:TestPoint TP5
-U 1 1 5FAFD167
-P 3400 7550
-F 0 "TP5" H 3458 7668 50  0000 L CNN
-F 1 " " H 3458 7577 50  0000 L CNN
-F 2 "TestPoint:TestPoint_Pad_D1.0mm" H 3600 7550 50  0001 C CNN
-F 3 "~" H 3600 7550 50  0001 C CNN
-	1    3400 7550
-	-1   0    0    1
-$EndComp
-Wire Wire Line
-	3400 7550 3400 7050
-Text Label 3400 7550 1    50   ~ 0
-MOTOR_PWM
 NoConn ~ 6800 3300
 $EndSCHEMATC
